File: DCMotor.kicad_sch (KiCad schematic)
At the start: 18 parts, among them J11 Conn_01x03_Socket, J12 Conn_01x03_Socket, J13 Conn_01x03_Socket, J14 Conn_01x03_Socket, J15 Conn_01x03_Socket, J6 Conn_01x02_Socket, J7 Conn_01x02_Socket, J8 Conn_01x02_Socket

Commit message: CircuitComplete
Parts:
- renumbered J12 to J10, J8 to J11, J13 to J12, J14 to J13, J15 to J14, J6 to J7, J11 to J8, J7 to J9, R28 to R27, R27 to R28
Connections:
- net VCC renamed +BATT

Commit message: before elimination of J7
Parts:
- renumbered R27 to R26, R28 to R27, R29 to R28, R30 to R29, R31 to R30, R32 to R31, R33 to R32, R34 to R33, R35 to R34, R36 to R35
Changed lines of the file:
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@@
 		(dnp no)
 		(fields_autoplaced yes)
-		(property "Reference" "R34"
+		(property "Reference" "R33"
 			(at 171.45 52.07 90)
 			(effects
@@
 			(project "chibarobo_board_2024"
 				(path "/7933aef9-9608-4ce1-b0d8-a4ffd3b998e4/10a4ce65-96c0-4b0e-ad7d-0749d3a88abd"
-					(reference "R34")
+					(reference "R33")
 					(unit 1)
 				)
@@
 		(dnp no)
 		(fields_autoplaced yes)
-		(property "Reference" "#PWR055"
+		(property "Reference" "#PWR054"
 			(at 72.39 49.53 0)
 			(effects
@@
 			(project "chibarobo_board_2024"
 				(path "/7933aef9-9608-4ce1-b0d8-a4ffd3b998e4/10a4ce65-96c0-4b0e-ad7d-0749d3a88abd"
-					(reference "#PWR055")
+					(reference "#PWR054")
 					(unit 1)
 				)
@@
 		(dnp no)
 		(fields_autoplaced yes)
-		(property "Reference" "#PWR052"
+		(property "Reference" "#PWR051"
 			(at 40.64 49.53 0)
 			(effects
@@
 			(project ""
 				(path "/7933aef9-9608-4ce1-b0d8-a4ffd3b998e4/10a4ce65-96c0-4b0e-ad7d-0749d3a88abd"
-					(reference "#PWR052")
+					(reference "#PWR051")
 					(unit 1)
 				)
@@
 		(dnp no)
 		(fields_autoplaced yes)
-		(property "Reference" "#PWR051"
+		(property "Reference" "#PWR050"
 			(at 40.64 45.72 0)
 			(effects
@@
 			(project ""
 				(path "/7933aef9-9608-4ce1-b0d8-a4ffd3b998e4/10a4ce65-96c0-4b0e-ad7d-0749d3a88abd"
-					(reference "#PWR051")
+					(reference "#PWR050")
 					(unit 1)
 				)
@@
 		(dnp no)
 		(fields_autoplaced yes)
-		(property "Reference" "R32"
+		(property "Reference" "R31"
 			(at 125.73 52.07 90)
 			(effects
@@
 			(project "chibarobo_board_2024"
 				(path "/7933aef9-9608-4ce1-b0d8-a4ffd3b998e4/10a4ce65-96c0-4b0e-ad7d-0749d3a88abd"
-					(reference "R32")
+					(reference "R31")
 					(unit 1)
 				)
@@
 		(dnp no)
 		(fields_autoplaced yes)
-		(property "Reference" "R31"
+		(property "Reference" "R30"
 			(at 125.73 49.53 90)
 			(effects
@@
 			(project "chibarobo_board_2024"
 				(path "/7933aef9-9608-4ce1-b0d8-a4ffd3b998e4/10a4ce65-96c0-4b0e-ad7d-0749d3a88abd"
-					(reference "R31")
+					(reference "R30")
 					(unit 1)
 				)
@@
 		(dnp no)
 		(fields_autoplaced yes)
-		(property "Reference" "R36"
+		(property "Reference" "R35"
 			(at 215.9 52.07 90)
 			(effects
@@
 			(project "chibarobo_board_2024"
 				(path "/7933aef9-9608-4ce1-b0d8-a4ffd3b998e4/10a4ce65-96c0-4b0e-ad7d-0749d3a88abd"
-					(reference "R36")
+					(reference "R35")
 					(unit 1)
 				)
@@
 		(dnp no)
 		(fields_autoplaced yes)
-		(property "Reference" "R33"
+		(property "Reference" "R32"
 			(at 171.45 49.53 90)
 			(effects
@@
 			(project "chibarobo_board_2024"
 				(path "/7933aef9-9608-4ce1-b0d8-a4ffd3b998e4/10a4ce65-96c0-4b0e-ad7d-0749d3a88abd"
-					(reference "R33")
+					(reference "R32")
 					(unit 1)
 				)
@@
 		(dnp no)
 		(fields_autoplaced yes)
-		(property "Reference" "R30"
+		(property "Reference" "R29"
 			(at 78.74 52.07 90)
 			(effects
@@
 			(project "chibarobo_board_2024"
 				(path "/7933aef9-9608-4ce1-b0d8-a4ffd3b998e4/10a4ce65-96c0-4b0e-ad7d-0749d3a88abd"
-					(reference "R30")
+					(reference "R29")
 					(unit 1)
 				)
@@
 		(dnp no)
 		(fields_autoplaced yes)
-		(property "Reference" "R35"
+		(property "Reference" "R34"
 			(at 215.9 49.53 90)
 			(effects
@@
 			(project "chibarobo_board_2024"
 				(path "/7933aef9-9608-4ce1-b0d8-a4ffd3b998e4/10a4ce65-96c0-4b0e-ad7d-0749d3a88abd"
-					(reference "R35")
+					(reference "R34")
 					(unit 1)
 				)
@@
 		(dnp no)
 		(fields_autoplaced yes)
-		(property "Reference" "#PWR057"
+		(property "Reference" "#PWR056"
 			(at 102.87 45.72 0)
 			(effects
@@
 			(project ""
 				(path "/7933aef9-9608-4ce1-b0d8-a4ffd3b998e4/10a4ce65-96c0-4b0e-ad7d-0749d3a88abd"
-					(reference "#PWR057")
+					(reference "#PWR056")
 					(unit 1)
 				)
@@
 		(dnp no)
 		(fields_autoplaced yes)
-		(property "Reference" "#PWR060"
+		(property "Reference" "#PWR059"
 			(at 179.07 67.31 0)
 			(effects
@@
 			(project "chibarobo_board_2024"
 				(path "/7933aef9-9608-4ce1-b0d8-a4ffd3b998e4/10a4ce65-96c0-4b0e-ad7d-0749d3a88abd"
-					(reference "#PWR060")
+					(reference "#PWR059")
 					(unit 1)
 				)
@@
 		(dnp no)
 		(fields_autoplaced yes)
-		(property "Reference" "#PWR058"
+		(property "Reference" "#PWR057"
 			(at 102.87 49.53 0)
 			(effects
@@
 			(project "chibarobo_board_2024"
 				(path "/7933aef9-9608-4ce1-b0d8-a4ffd3b998e4/10a4ce65-96c0-4b0e-ad7d-0749d3a88abd"
-					(reference "#PWR058")
+					(reference "#PWR057")
 					(unit 1)
 				)
@@
 		(dnp no)
 		(fields_autoplaced yes)
-		(property "Reference" "#PWR054"
+		(property "Reference" "#PWR053"
 			(at 72.39 45.72 0)
 			(effects
@@
 			(project ""
 				(path "/7933aef9-9608-4ce1-b0d8-a4ffd3b998e4/10a4ce65-96c0-4b0e-ad7d-0749d3a88abd"
-					(reference "#PWR054")
+					(reference "#PWR053")
 					(unit 1)
 				)
@@
 		(dnp no)
 		(fields_autoplaced yes)
-		(property "Reference" "#PWR056"
+		(property "Reference" "#PWR055"
 			(at 86.36 67.31 0)
 			(effects
@@
 			(project "chibarobo_board_2024"
 				(path "/7933aef9-9608-4ce1-b0d8-a4ffd3b998e4/10a4ce65-96c0-4b0e-ad7d-0749d3a88abd"
-					(reference "#PWR056")
+					(reference "#PWR055")
 					(unit 1)
 				)
@@
 		(dnp no)
 		(fields_autoplaced yes)
-		(property "Reference" "#PWR061"
+		(property "Reference" "#PWR060"
 			(at 223.52 67.31 0)
 			(effects
@@
 			(project "chibarobo_board_2024"
 				(path "/7933aef9-9608-4ce1-b0d8-a4ffd3b998e4/10a4ce65-96c0-4b0e-ad7d-0749d3a88abd"
-					(reference "#PWR061")
+					(reference "#PWR060")
 					(unit 1)
 				)
@@
 		(dnp no)
 		(fields_autoplaced yes)
-		(property "Reference" "#PWR053"
+		(property "Reference" "#PWR052"
 			(at 40.64 67.31 0)
 			(effects
@@
 			(project ""
 				(path "/7933aef9-9608-4ce1-b0d8-a4ffd3b998e4/10a4ce65-96c0-4b0e-ad7d-0749d3a88abd"
-					(reference "#PWR053")
+					(reference "#PWR052")
 					(unit 1)
 				)
@@
 		(dnp no)
 		(fields_autoplaced yes)
-		(property "Reference" "R27"
+		(property "Reference" "R26"
 			(at 33.02 49.53 90)
 			(effects
@@
 			(project ""
 				(path "/7933aef9-9608-4ce1-b0d8-a4ffd3b998e4/10a4ce65-96c0-4b0e-ad7d-0749d3a88abd"
-					(reference "R27")
+					(reference "R26")
 					(unit 1)
 				)
@@
 		(dnp no)
 		(fields_autoplaced yes)
-		(property "Reference" "R29"
+		(property "Reference" "R28"
 			(at 78.74 49.53 90)
 			(effects
@@
 			(project "chibarobo_board_2024"
 				(path "/7933aef9-9608-4ce1-b0d8-a4ffd3b998e4/10a4ce65-96c0-4b0e-ad7d-0749d3a88abd"
-					(reference "R29")
+					(reference "R28")
 					(unit 1)
 				)
@@
 		(dnp no)
 		(fields_autoplaced yes)
-		(property "Reference" "R28"
+		(property "Reference" "R27"
 			(at 33.02 52.07 90)
 			(effects
@@
 			(project ""
 				(path "/7933aef9-9608-4ce1-b0d8-a4ffd3b998e4/10a4ce65-96c0-4b0e-ad7d-0749d3a88abd"
-					(reference "R28")
+					(reference "R27")
 					(unit 1)
 				)
@@
 		(dnp no)
 		(fields_autoplaced yes)
-		(property "Reference" "#PWR059"
+		(property "Reference" "#PWR058"
 			(at 133.35 67.31 0)
 			(effects
@@
 			(project "chibarobo_board_2024"
 				(path "/7933aef9-9608-4ce1-b0d8-a4ffd3b998e4/10a4ce65-96c0-4b0e-ad7d-0749d3a88abd"
-					(reference "#PWR059")
-					(unit 1)
-				)
+					(reference "#PWR058")
+					(unit 1)
+				)

Commit message: Rev1.2
Parts:
- removed J7: Conn_01x02_Socket, Connector_AMASS:AMASS_XT60-F_1x02_P7.20mm_Vertical, symbol Connector:Conn_01x02_Socket
- renumbered J11 to J10, J12 to J11, J13 to J12, J14 to J13, J8 to J7, J9 to J8, J10 to J9
Changed lines of the file:
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@@
 		(dnp no)
 		(fields_autoplaced yes)
-		(property "Reference" "#PWR054"
+		(property "Reference" "#PWR053"
 			(at 72.39 49.53 0)
 			(effects
@@
 			(project "chibarobo_board_2024"
 				(path "/7933aef9-9608-4ce1-b0d8-a4ffd3b998e4/10a4ce65-96c0-4b0e-ad7d-0749d3a88abd"
-					(reference "#PWR054")
-					(unit 1)
-				)
-			)
-		)
-	)
-	(symbol
-		(lib_id "power:GNDPWR")
-		(at 40.64 44.45 0)
-		(unit 1)
-		(exclude_from_sim no)
-		(in_bom yes)
-		(on_board yes)
-		(dnp no)
-		(fields_autoplaced yes)
-		(property "Reference" "#PWR051"
-			(at 40.64 49.53 0)
-			(effects
-				(font
-					(size 1.27 1.27)
-				)
-				(hide yes)
-			)
-		)
-		(property "Value" "GNDPWR"
-			(at 40.513 48.26 0)
-			(effects
-				(font
-					(size 1.27 1.27)
-				)
-			)
-		)
-		(property "Footprint" ""
-			(at 40.64 45.72 0)
-			(effects
-				(font
-					(size 1.27 1.27)
-				)
-				(hide yes)
-			)
-		)
-		(property "Datasheet" ""
-			(at 40.64 45.72 0)
-			(effects
-				(font
-					(size 1.27 1.27)
-				)
-				(hide yes)
-			)
-		)
-		(property "Description" "Power symbol creates a global label with name \"GNDPWR\" , global ground"
-			(at 40.64 44.45 0)
-			(effects
-				(font
-					(size 1.27 1.27)
-				)
-				(hide yes)
-			)
-		)
-		(pin "1"
-		)
-		(instances
-			(project ""
-				(path "/7933aef9-9608-4ce1-b0d8-a4ffd3b998e4/10a4ce65-96c0-4b0e-ad7d-0749d3a88abd"
-					(reference "#PWR051")
+					(reference "#PWR053")
 					(unit 1)
 				)
@@
 		(on_board yes)
 		(dnp no)
-		(property "Reference" "J11"
+		(property "Reference" "J10"
 			(at 109.22 44.4501 0)
 			(effects
@@
 			(project "chibarobo_board_2024"
 				(path "/7933aef9-9608-4ce1-b0d8-a4ffd3b998e4/10a4ce65-96c0-4b0e-ad7d-0749d3a88abd"
-					(reference "J11")
+					(reference "J10")
 					(unit 1)
 				)
@@
 		(on_board yes)
 		(dnp no)
-		(property "Reference" "J13"
+		(property "Reference" "J12"
 			(at 185.42 59.6901 0)
 			(effects
@@
 			(project "chibarobo_board_2024"
 				(path "/7933aef9-9608-4ce1-b0d8-a4ffd3b998e4/10a4ce65-96c0-4b0e-ad7d-0749d3a88abd"
-					(reference "J13")
-					(unit 1)
-				)
-			)
-		)
-	)
-	(symbol
-		(lib_id "power:+BATT")
-		(at 40.64 41.91 0)
-		(unit 1)
-		(exclude_from_sim no)
-		(in_bom yes)
-		(on_board yes)
-		(dnp no)
-		(fields_autoplaced yes)
-		(property "Reference" "#PWR050"
-			(at 40.64 45.72 0)
-			(effects
-				(font
-					(size 1.27 1.27)
-				)
-				(hide yes)
-			)
-		)
-		(property "Value" "+BATT"
-			(at 40.64 36.83 0)
-			(effects
-				(font
-					(size 1.27 1.27)
-				)
-			)
-		)
-		(property "Footprint" ""
-			(at 40.64 41.91 0)
-			(effects
-				(font
-					(size 1.27 1.27)
-				)
-				(hide yes)
-			)
-		)
-		(property "Datasheet" ""
-			(at 40.64 41.91 0)
-			(effects
-				(font
-					(size 1.27 1.27)
-				)
-				(hide yes)
-			)
-		)
-		(property "Description" "Power symbol creates a global label with name \"+BATT\""
-			(at 40.64 41.91 0)
-			(effects
-				(font
-					(size 1.27 1.27)
-				)
-				(hide yes)
-			)
-		)
-		(pin "1"
-		)
-		(instances
-			(project ""
-				(path "/7933aef9-9608-4ce1-b0d8-a4ffd3b998e4/10a4ce65-96c0-4b0e-ad7d-0749d3a88abd"
-					(reference "#PWR050")
+					(reference "J12")
 					(unit 1)
 				)
@@
 		(on_board yes)
 		(dnp no)
-		(property "Reference" "J8"
+		(property "Reference" "J7"
 			(at 46.99 59.6901 0)
 			(effects
@@
 			(project ""
 				(path "/7933aef9-9608-4ce1-b0d8-a4ffd3b998e4/10a4ce65-96c0-4b0e-ad7d-0749d3a88abd"
-					(reference "J8")
+					(reference "J7")
 					(unit 1)
 				)
@@
 		(on_board yes)
 		(dnp no)
-		(property "Reference" "J12"
+		(property "Reference" "J11"
 			(at 139.7 59.6901 0)
 			(effects
@@
 			(project "chibarobo_board_2024"
 				(path "/7933aef9-9608-4ce1-b0d8-a4ffd3b998e4/10a4ce65-96c0-4b0e-ad7d-0749d3a88abd"
-					(reference "J12")
+					(reference "J11")
 					(unit 1)
 				)
@@
 		(on_board yes)
 		(dnp no)
-		(property "Reference" "J9"
+		(property "Reference" "J8"
 			(at 78.74 44.4501 0)
 			(effects
@@
 			(project "chibarobo_board_2024"
 				(path "/7933aef9-9608-4ce1-b0d8-a4ffd3b998e4/10a4ce65-96c0-4b0e-ad7d-0749d3a88abd"
-					(reference "J9")
+					(reference "J8")
 					(unit 1)
 				)
@@
 	)
 	(symbol
-		(lib_id "Connector:Conn_01x02_Socket")
-		(at 45.72 44.45 0)
-		(mirror x)
-		(unit 1)
-		(exclude_from_sim no)
-		(in_bom yes)
-		(on_board yes)
-		(dnp no)
-		(property "Reference" "J7"
-			(at 46.99 44.4501 0)
-			(effects
-				(font
-					(size 1.27 1.27)
-				)
-				(justify left)
-			)
-		)
-		(property "Value" "Conn_01x02_Socket"
-			(at 46.99 41.9101 0)
-			(effects
-				(font
-					(size 1.27 1.27)
-				)
-				(justify left)
-			)
-		)
-		(property "Footprint" "Connector_AMASS:AMASS_XT60-F_1x02_P7.20mm_Vertical"
-			(at 45.72 44.45 0)
-			(effects
-				(font
-					(size 1.27 1.27)
-				)
-				(hide yes)
-			)
-		)
-		(property "Datasheet" "~"
-			(at 45.72 44.45 0)
-			(effects
-				(font
-					(size 1.27 1.27)
-				)
-				(hide yes)
-			)
-		)
-		(property "Description" "Generic connector, single row, 01x02, script generated"
-			(at 45.72 44.45 0)
-			(effects
-				(font
-					(size 1.27 1.27)
-				)
-				(hide yes)
-			)
-		)
-		(property "JLCPCB Parts#" ""
-			(at 45.72 44.45 0)
-			(effects
-				(font
-					(size 1.27 1.27)
-				)
-				(hide yes)
-			)
-		)
-		(pin "2"
-		)
-		(pin "1"
-		)
-		(instances
-			(project ""
-				(path "/7933aef9-9608-4ce1-b0d8-a4ffd3b998e4/10a4ce65-96c0-4b0e-ad7d-0749d3a88abd"
-					(reference "J7")
-					(unit 1)
-				)
-			)
-		)
-	)
-	(symbol
 		(lib_id "Device:R")
 		(at 78.74 58.42 90)
@@
 		(dnp no)
 		(fields_autoplaced yes)
-		(property "Reference" "#PWR056"
+		(property "Reference" "#PWR055"
 			(at 102.87 45.72 0)
 			(effects
@@
 			(project ""
 				(path "/7933aef9-9608-4ce1-b0d8-a4ffd3b998e4/10a4ce65-96c0-4b0e-ad7d-0749d3a88abd"
-					(reference "#PWR056")
+					(reference "#PWR055")
 					(unit 1)
 				)
@@
 		(dnp no)
 		(fields_autoplaced yes)
-		(property "Reference" "#PWR059"
+		(property "Reference" "#PWR058"
 			(at 179.07 67.31 0)
 			(effects
@@
 			(project "chibarobo_board_2024"
 				(path "/7933aef9-9608-4ce1-b0d8-a4ffd3b998e4/10a4ce65-96c0-4b0e-ad7d-0749d3a88abd"
-					(reference "#PWR059")
+					(reference "#PWR058")
 					(unit 1)
 				)
@@
 		(dnp no)
 		(fields_autoplaced yes)
-		(property "Reference" "#PWR057"
+		(property "Reference" "#PWR056"
 			(at 102.87 49.53 0)
 			(effects
@@
 			(project "chibarobo_board_2024"
 				(path "/7933aef9-9608-4ce1-b0d8-a4ffd3b998e4/10a4ce65-96c0-4b0e-ad7d-0749d3a88abd"
-					(reference "#PWR057")
+					(reference "#PWR056")
 					(unit 1)
 				)
@@
 		(dnp no)
 		(fields_autoplaced yes)
-		(property "Reference" "#PWR053"
+		(property "Reference" "#PWR052"
 			(at 72.39 45.72 0)
 			(effects
@@
 			(project ""
 				(path "/7933aef9-9608-4ce1-b0d8-a4ffd3b998e4/10a4ce65-96c0-4b0e-ad7d-0749d3a88abd"
-					(reference "#PWR053")
+					(reference "#PWR052")
 					(unit 1)
 				)
@@
 		(dnp no)
 		(fields_autoplaced yes)
-		(property "Reference" "#PWR055"
+		(property "Reference" "#PWR054"
 			(at 86.36 67.31 0)
 			(effects
@@
 			(project "chibarobo_board_2024"
 				(path "/7933aef9-9608-4ce1-b0d8-a4ffd3b998e4/10a4ce65-96c0-4b0e-ad7d-0749d3a88abd"
-					(reference "#PWR055")
+					(reference "#PWR054")
 					(unit 1)
 				)
@@
 		(dnp no)
 		(fields_autoplaced yes)
-		(property "Reference" "#PWR060"
+		(property "Reference" "#PWR059"
 			(at 223.52 67.31 0)
 			(effects
@@
 			(project "chibarobo_board_2024"
 				(path "/7933aef9-9608-4ce1-b0d8-a4ffd3b998e4/10a4ce65-96c0-4b0e-ad7d-0749d3a88abd"
-					(reference "#PWR060")
+					(reference "#PWR059")
 					(unit 1)
 				)
@@
 		(dnp no)
 		(fields_autoplaced yes)
-		(property "Reference" "#PWR052"
+		(property "Reference" "#PWR051"
 			(at 40.64 67.31 0)
 			(effects
@@
 			(project ""
 				(path "/7933aef9-9608-4ce1-b0d8-a4ffd3b998e4/10a4ce65-96c0-4b0e-ad7d-0749d3a88abd"
-					(reference "#PWR052")
+					(reference "#PWR051")
 					(unit 1)
 				)
@@
 		(on_board yes)
 		(dnp no)
-		(property "Reference" "J14"
+		(property "Reference" "J13"
 			(at 229.87 59.6901 0)
 			(effects
@@
 			(project "chibarobo_board_2024"
 				(path "/7933aef9-9608-4ce1-b0d8-a4ffd3b998e4/10a4ce65-96c0-4b0e-ad7d-0749d3a88abd"
-					(reference "J14")
+					(reference "J13")
 					(unit 1)
 				)
@@
 		(on_board yes)
 		(dnp no)
-		(property "Reference" "J10"
+		(property "Reference" "J9"
 			(at 92.71 59.6901 0)
 			(effects
@@
 			(project "chibarobo_board_2024"
 				(path "/7933aef9-9608-4ce1-b0d8-a4ffd3b998e4/10a4ce65-96c0-4b0e-ad7d-0749d3a88abd"
-					(reference "J10")
+					(reference "J9")
 					(unit 1)
 				)
@@
 		(dnp no)
 		(fields_autoplaced yes)
-		(property "Reference" "#PWR058"
+		(property "Reference" "#PWR057"
 			(at 133.35 67.31 0)
 			(effects
@@
 			(project "chibarobo_board_2024"
 				(path "/7933aef9-9608-4ce1-b0d8-a4ffd3b998e4/10a4ce65-96c0-4b0e-ad7d-0749d3a88abd"
-					(reference "#PWR058")
-					(unit 1)
-				)
+					(reference "#PWR057")
+					(unit 1)
+				)
