File: EMS.kicad_sch (KiCad schematic)
At the start: 31 parts, among them IC5 TC7W14FK, J16 Conn_01x02_Socket, Q10 2SC2712-GR_TE85L,F, Q8 2SA1162-GR_F_, Q9 2SC2712-GR_TE85L,F, U8 TLP291

Commit message: Rev1.2
Parts:
- renumbered J16 to J15
