File: MainSwitch.kicad_sch (KiCad schematic)
At the start: 9 parts, among them K1 V23134J, Q13 2SC2712-GR_TE85L,F, Q14 BUZ11

Commit message: Rev1
Parts:
- removed Q14: BUZ11, Package_TO_SOT_THT:TO-220-3_Vertical, symbol Transistor_FET:BUZ11
- added Q14: IRFL014TRPBF, SamacSys_Parts:SOT230P700X180-4N, symbol SamacSys_Parts:IRFL014TRPBF
- D8: footprint Diode_THT:D_5W_P10.16mm_Horizontal -> Diode_THT:D_5W_P5.08mm_Vertical_KathodeUp
Connections:
- net +BATT: no longer R60.1
- net -BATT: now also Q14.3 (S)
- net at C19.1, D9.1 (K), R61.1: now also Q14.1 (G)
- net at D8.2 (A), K1.85: now also Q14.2 (D_1), Q14.4 (D_2)
- new net SAFE_+BATT: R60.1
Other:
- moved on the sheet: C19, D9, R61

Commit message: Rev1
Parts:
- D9: JLCPCB Parts# (none) -> C19077447
- Q13: JLCPCB Parts# (none) -> C83447
- Q14: JLCPCB Parts# (none) -> C428746

Commit message: before elimination of J7
Parts:
- renumbered D8 to D10, Q13 to Q14, Q14 to Q15, R59 to R58, R60 to R59, R61 to R60
