File: PowerSupply.kicad_sch (KiCad schematic)
At the start: 2 parts, among them IC2 D44H8, Q11 2SC2712-GR_TE85L,F

Commit message: CircuitComplete
Parts:
- removed IC2: D44H8, TO270P460X1020X2008-3P, symbol SamacSys_Parts:D44H8
- removed Q11: 2SC2712-GR_TE85L,F, SOT95P260X156-3N, symbol SamacSys_Parts:2SC2712-GR_TE85L,F
- added C10, C11, C13: 100n, Capacitor_SMD:C_0603_1608Metric, symbol Device:C
- added C12: 10u, Capacitor_THT:CP_Radial_D5.0mm_P2.00mm, symbol Device:C_Polarized
- added C9: 1u, Capacitor_SMD:C_0603_1608Metric, symbol Device:C
- added D1, D3: NSI50010YT1G, Diode_SMD:D_SOD-123, symbol Device:D_Constant_Current
- added D2: VLMKG3400, LED_SMD:LED_Avago_PLCC4_3.2x2.8mm_CW, symbol Device:LED_Dual_KAKA
- added F1: Fuse, Fuse:Fuse_1206_3216Metric, symbol Device:Fuse
- added IC3: TC74HC00AF_F_, SamacSys_Parts:SOIC127P780X190-14N, symbol SamacSys_Parts:TC74HC00AF_F_
- added IC4: L78M05CDT, SamacSys_Parts:TO225P972X240-3N, symbol SamacSys_Parts:L78M05CDT
- added J16: Conn_01x02_Socket, original:AMASS_XT90PW-M_1x02_P11.00mm_Horizontal, symbol Connector:Conn_01x02_Socket
- added R37: 200k, Resistor_SMD:R_0603_1608Metric, symbol Device:R
- added R38, R39: 2.2k, Resistor_SMD:R_0603_1608Metric, symbol Device:R
- added U6: 74LVC1G123, Package_SO:VSSOP-8_2.3x2mm_P0.5mm, symbol 74xGxx:74LVC1G123
Connections:
- new net: IC3.10 (3B), IC3.11 (4Y), IC3.9 (3A)
- new net: IC3.13 (4B), IC3.3 (1Y)
- new net: C9.1, R37.2, U6.7 (RCext)
- new net: C12.1, D2.2 (K1), D2.4 (K2), F1.1, IC4.1 (IN)
- new net: D2.3 (A2), D3.2 (A)
- new net: D1.2 (A), D2.1 (A1)
- new net: R38.2, U6.3 (~{CLR})
- new net: R39.1, U6.5 (Q)
- new net +BATT: F1.2, J16.2 (Pin_2)
- new net -BATT: C10.2, C11.2, C12.2, C13.2, C9.2, D1.1 (K), IC3.7 (GND), IC4.3 (GND), J16.1 (Pin_1), U6.1 (~{A}), U6.4 (GND), U6.6 (Cext)
- new net GNDPWR: D3.1 (K)
- new net LOGPWR: C10.1, C11.1, C13.1, IC3.14 (VCC), IC4.2 (OUT), R37.1, R38.1, U6.8 (VCC)
- new net MS: IC3.8 (3Y)
- new net WMUP: IC3.1 (1A), IC3.2 (1B), IC3.5 (2B), R39.2
- new net ~{EMS}: IC3.12 (4A), IC3.4 (2A), U6.2 (B)
- new net ~{SS}: IC3.6 (2Y)
Other:
- added sheet MainSwitch (MainSwitch.kicad_sch)
- added sheet SoftStart (SoftStart.kicad_sch)
- sheet EMS ports: added LOGPWR; removed none

Commit message: Rev1
Parts:
- removed C12: 10u, Capacitor_THT:CP_Radial_D5.0mm_P2.00mm, symbol Device:C_Polarized
- added C12: 10u, Capacitor_SMD:C_0805_2012Metric, symbol Device:C
Connections:
- net -BATT: now also C12.2
- net SAFE_+BATT: now reaches D2.2 (K1), D2.4 (K2), F1.1, IC4.1 (IN)
- net SAFE_+BATT: now also C12.1
Other:
- sheet MainSwitch ports: added SAFE_+BATT; removed none
- sheet SoftStart ports: added SAFE_+BATT; removed LOGPWR
Changed lines of the file:
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@@
 	)
 	(junction
-		(at 49.53 114.3)
+		(at 160.02 123.19)
 		(diameter 0)
 		(color 0 0 0 0)
 	)
 	(junction
-		(at 157.48 39.37)
+		(at 49.53 114.3)
 		(diameter 0)
 		(color 0 0 0 0)
 	)
 	(junction
-		(at 64.77 54.61)
+		(at 157.48 39.37)
 		(diameter 0)
 		(color 0 0 0 0)
@@
 	(wire
 		(pts
+			(xy 165.1 127) (xy 160.02 127)
+		)
+		(stroke
+			(width 0)
+			(type default)
+		)
+	)
+	(wire
+		(pts
 			(xy 177.8 39.37) (xy 175.26 39.37)
 		)
@@
 	(wire
 		(pts
-			(xy 64.77 73.66) (xy 60.96 73.66)
+			(xy 64.77 76.2) (xy 60.96 76.2)
 		)
 		(stroke
@@
 	(wire
 		(pts
+			(xy 160.02 127) (xy 160.02 123.19)
+		)
+		(stroke
+			(width 0)
+			(type default)
+		)
+	)
+	(wire
+		(pts
 			(xy 36.83 109.22) (xy 38.1 109.22)
 		)
@@
 	(wire
 		(pts
+			(xy 60.96 73.66) (xy 63.5 73.66)
+		)
+		(stroke
+			(width 0)
+			(type default)
+		)
+	)
+	(wire
+		(pts
 			(xy 120.65 113.03) (xy 120.65 87.63)
 		)
@@
 	(wire
 		(pts
-			(xy 60.96 54.61) (xy 64.77 54.61)
+			(xy 162.56 69.85) (xy 162.56 74.93)
 		)
 		(stroke
@@
 	(wire
 		(pts
-			(xy 162.56 69.85) (xy 162.56 74.93)
+			(xy 160.02 113.03) (xy 165.1 113.03)
 		)
 		(stroke
@@
 	(wire
 		(pts
-			(xy 160.02 113.03) (xy 165.1 113.03)
+			(xy 64.77 39.37) (xy 72.39 39.37)
 		)
 		(stroke
@@
 	(wire
 		(pts
-			(xy 64.77 39.37) (xy 72.39 39.37)
+			(xy 49.53 114.3) (xy 54.61 114.3)
 		)
 		(stroke
@@
 	(wire
 		(pts
-			(xy 49.53 114.3) (xy 54.61 114.3)
+			(xy 60.96 54.61) (xy 63.5 54.61)
 		)
 		(stroke
@@
 	(wire
 		(pts
-			(xy 64.77 39.37) (xy 64.77 54.61)
+			(xy 64.77 39.37) (xy 64.77 76.2)
 		)
 		(stroke
@@
 	(wire
 		(pts
-			(xy 60.96 77.47) (xy 63.5 77.47)
+			(xy 60.96 78.74) (xy 63.5 78.74)
 		)
 		(stroke
@@
 		)
 	)
-	(wire
-		(pts
-			(xy 64.77 54.61) (xy 64.77 73.66)
-		)
-		(stroke
-			(width 0)
-			(type default)
-		)
-	)
 	(label "~{SS}"
 		(at 63.5 58.42 0)
@@
 	)
 	(label "MS"
-		(at 63.5 77.47 0)
+		(at 63.5 78.74 0)
 		(fields_autoplaced yes)
 		(effects
@@
 		)
 	)
+	(label "SAFE_+BATT"
+		(at 162.56 39.37 0)
+		(fields_autoplaced yes)
+		(effects
+			(font
+				(size 1.27 1.27)
+			)
+			(justify left bottom)
+		)
+	)
 	(label "~{SS}"
 		(at 128.27 120.65 180)
@@
 		)
 	)
+	(label "SAFE_+BATT"
+		(at 63.5 54.61 0)
+		(fields_autoplaced yes)
+		(effects
+			(font
+				(size 1.27 1.27)
+			)
+			(justify left bottom)
+		)
+	)
 	(label "~{EMS}"
 		(at 63.5 43.18 0)
@@
 		)
 	)
+	(label "SAFE_+BATT"
+		(at 63.5 73.66 0)
+		(fields_autoplaced yes)
+		(effects
+			(font
+				(size 1.27 1.27)
+			)
+			(justify left bottom)
+		)
+	)
 	(label "LOGPWR"
 		(at 26.67 100.33 0)
@@
 		)
 	)
+	(global_label "MS"
+		(shape output)
+		(at 165.1 127 0)
+		(fields_autoplaced yes)
+		(effects
+			(font
+				(size 1.27 1.27)
+			)
+			(justify left)
+		)
+		(property "Intersheetrefs" "${INTERSHEET_REFS}"
+			(at 170.7461 127 0)
+			(effects
+				(font
+					(size 1.27 1.27)
+				)
+				(justify left)
+				(hide yes)
+			)
+		)
+	)
 	(symbol
 		(lib_id "power:-BATT")
@@
 	)
 	(symbol
-		(lib_id "Device:C_Polarized")
-		(at 151.13 45.72 0)
-		(unit 1)
-		(exclude_from_sim no)
-		(in_bom yes)
-		(on_board yes)
-		(dnp no)
-		(fields_autoplaced yes)
-		(property "Reference" "C12"
-			(at 154.94 43.5609 0)
-			(effects
-				(font
-					(size 1.27 1.27)
-				)
-				(justify left)
-			)
-		)
-		(property "Value" "10u"
-			(at 154.94 46.1009 0)
-			(effects
-				(font
-					(size 1.27 1.27)
-				)
-				(justify left)
-			)
-		)
-		(property "Footprint" "Capacitor_THT:CP_Radial_D5.0mm_P2.00mm"
-			(at 152.0952 49.53 0)
-			(effects
-				(font
-					(size 1.27 1.27)
-				)
-				(hide yes)
-			)
-		)
-		(property "Datasheet" "~"
-			(at 151.13 45.72 0)
-			(effects
-				(font
-					(size 1.27 1.27)
-				)
-				(hide yes)
-			)
-		)
-		(property "Description" "Polarized capacitor"
-			(at 151.13 45.72 0)
-			(effects
-				(font
-					(size 1.27 1.27)
-				)
-				(hide yes)
-			)
-		)
-		(pin "2"
-		)
-		(pin "1"
-		)
-		(instances
-			(project ""
-				(path "/7933aef9-9608-4ce1-b0d8-a4ffd3b998e4/a3ca3e3d-7f11-4e5a-900e-b192a8343e04"
-					(reference "C12")
-					(unit 1)
-				)
-			)
-		)
-	)
-	(symbol
 		(lib_id "Device:D_Constant_Current")
 		(at 162.56 66.04 90)
@@
 	)
 	(symbol
+		(lib_id "Device:C")
+		(at 151.13 45.72 0)
+		(unit 1)
+		(exclude_from_sim no)
+		(in_bom yes)
+		(on_board yes)
+		(dnp no)
+		(fields_autoplaced yes)
+		(property "Reference" "C12"
+			(at 154.94 44.4499 0)
+			(effects
+				(font
+					(size 1.27 1.27)
+				)
+				(justify left)
+			)
+		)
+		(property "Value" "10u"
+			(at 154.94 46.9899 0)
+			(effects
+				(font
+					(size 1.27 1.27)
+				)
+				(justify left)
+			)
+		)
+		(property "Footprint" "Capacitor_SMD:C_0805_2012Metric"
+			(at 152.0952 49.53 0)
+			(effects
+				(font
+					(size 1.27 1.27)
+				)
+				(hide yes)
+			)
+		)
+		(property "Datasheet" "~"
+			(at 151.13 45.72 0)
+			(effects
+				(font
+					(size 1.27 1.27)
+				)
+				(hide yes)
+			)
+		)
+		(property "Description" "Unpolarized capacitor"
+			(at 151.13 45.72 0)
+			(effects
+				(font
+					(size 1.27 1.27)
+				)
+				(hide yes)
+			)
+		)
+		(pin "2"
+		)
+		(pin "1"
+		)
+		(instances
+			(project ""
+				(path "/7933aef9-9608-4ce1-b0d8-a4ffd3b998e4/a3ca3e3d-7f11-4e5a-900e-b192a8343e04"
+					(reference "C12")
+					(unit 1)
+				)
+			)
+		)
+	)
+	(symbol
 		(lib_id "Device:R")
 		(at 88.9 106.68 90)
@@
 	(sheet
 		(at 27.94 68.58)
-		(size 33.02 12.7)
+		(size 33.02 13.97)
 		(fields_autoplaced yes)
 		(stroke
@@
 		)
 		(property "Sheetfile" "MainSwitch.kicad_sch"
-			(at 27.94 81.8646 0)
+			(at 27.94 83.1346 0)
 			(effects
 				(font
@@
 		)
 		(pin "MS" input
-			(at 60.96 77.47 0)
+			(at 60.96 78.74 0)
 			(effects
 				(font
@@
 		)
 		(pin "LOGPWR" input
+			(at 60.96 76.2 0)
+			(effects
+				(font
+					(size 1.27 1.27)
+				)
+				(justify right)
+			)
+		)
+		(pin "SAFE_+BATT" input
 			(at 60.96 73.66 0)
 			(effects
@@
 			)
 		)
-		(pin "LOGPWR" input
-			(at 60.96 54.61 0)
+		(pin "~{SS}" input
+			(at 60.96 58.42 0)
 			(effects
 				(font
@@
 			)
 		)
-		(pin "~{SS}" input
-			(at 60.96 58.42 0)
+		(pin "SAFE_+BATT" input
+			(at 60.96 54.61 0)
 			(effects
 				(font

Commit message: Rev1
Parts:
- IC4: JLCPCB Parts# (none) -> C55509
- U6: JLCPCB Parts# (none) -> C77273
Changed lines of the file:
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@@
+			)
+		)
+		(property "JLCPCB Parts#" ""
+			(at 134.62 107.95 0)
+			(effects
+				(font
+					(size 1.27 1.27)
+				)
+				(hide yes)
 			)
 		)
@@
 			)
 		)
+		(property "JLCPCB Parts#" ""
+			(at 43.18 109.22 0)
+			(effects
+				(font
+					(size 1.27 1.27)
+				)
+				(hide yes)
+			)
+		)
 		(pin "2"
 		)
@@
 			)
 		)
+		(property "JLCPCB Parts#" ""
+			(at 72.39 53.34 0)
+			(effects
+				(font
+					(size 1.27 1.27)
+				)
+				(hide yes)
+			)
+		)
 		(pin "1"
 		)
@@
 			)
 		)
+		(property "JLCPCB Parts#" ""
+			(at 162.56 66.04 0)
+			(effects
+				(font
+					(size 1.27 1.27)
+				)
+				(hide yes)
+			)
+		)
 		(pin "2"
 		)
@@
 			)
 		)
+		(property "JLCPCB Parts#" ""
+			(at 157.48 66.04 0)
+			(effects
+				(font
+					(size 1.27 1.27)
+				)
+				(hide yes)
+			)
+		)
 		(pin "2"
 		)
@@
 			)
 		)
+		(property "JLCPCB Parts#" " C77273"
+			(at 67.31 111.76 0)
+			(effects
+				(font
+					(size 1.27 1.27)
+				)
+				(hide yes)
+			)
+		)
 		(pin "3"
 		)
@@
 			)
 		)
+		(property "JLCPCB Parts#" ""
+			(at 105.41 45.72 0)
+			(effects
+				(font
+					(size 1.27 1.27)
+				)
+				(hide yes)
+			)
+		)
 		(pin "2"
 		)
@@
 			)
 		)
+		(property "JLCPCB Parts#" ""
+			(at 171.45 39.37 0)
+			(effects
+				(font
+					(size 1.27 1.27)
+				)
+				(hide yes)
+			)
+		)
 		(pin "1"
 		)
@@
 			)
 		)
+		(property "JLCPCB Parts#" ""
+			(at 46.99 129.54 0)
+			(effects
+				(font
+					(size 1.27 1.27)
+				)
+				(hide yes)
+			)
+		)
 		(pin "2"
 		)
@@
 			)
 		)
+		(property "JLCPCB Parts#" ""
+			(at 160.02 49.53 0)
+			(effects
+				(font
+					(size 1.27 1.27)
+				)
+				(hide yes)
+			)
+		)
 		(pin "3"
 		)
@@
 		)
 		(property "Description" "Resistor"
+			(at 33.02 109.22 0)
+			(effects
+				(font
+					(size 1.27 1.27)
+				)
+				(hide yes)
+			)
+		)
+		(property "JLCPCB Parts#" ""
 			(at 33.02 109.22 0)
 			(effects
@@
 			)
 		)
+		(property "JLCPCB Parts#" ""
+			(at 227.33 72.39 0)
+			(effects
+				(font
+					(size 1.27 1.27)
+				)
+				(hide yes)
+			)
+		)
 		(pin "2"
 		)
@@
 		)
 		(property "Description" "Unpolarized capacitor"
+			(at 165.1 99.06 0)
+			(effects
+				(font
+					(size 1.27 1.27)
+				)
+				(hide yes)
+			)
+		)
+		(property "JLCPCB Parts#" ""
 			(at 165.1 99.06 0)
 			(effects
@@
 			)
 		)
+		(property "JLCPCB Parts#" " C77273"
+			(at 83.82 54.61 0)
+			(effects
+				(font
+					(size 1.27 1.27)
+				)
+				(hide yes)
+			)
+		)
 		(pin "3"
 		)
@@
 			)
 		)
+		(property "JLCPCB Parts#" "C55509"
+			(at 146.05 39.37 0)
+			(effects
+				(font
+					(size 1.27 1.27)
+				)
+				(hide yes)
+			)
+		)
 		(pin "2"
 		)
@@
 			)
 		)
+		(property "JLCPCB Parts#" ""
+			(at 151.13 45.72 0)
+			(effects
+				(font
+					(size 1.27 1.27)
+				)
+				(hide yes)
+			)
+		)
 		(pin "2"
 		)
@@
 			(at 88.9 106.68 0)
 			(effects
+				(font
+					(size 1.27 1.27)
+				)
+				(hide yes)
+			)
+		)
+		(property "JLCPCB Parts#" ""
+			(at 88.9 106.68 0)
+			(effects

Commit message: before elimination of J7
Parts:
- renumbered J16 to J15, R37 to R36, R38 to R37, R39 to R38, U6 to U7
Connections:
- net -BATT: now also IC4.2 (GND); no longer IC4.3 (GND)
- net LOGPWR: now also IC4.3 (OUT); no longer IC4.2 (OUT)
Changed lines of the file:
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@@
 		(dnp no)
 		(fields_autoplaced yes)
-		(property "Reference" "#PWR069"
+		(property "Reference" "#PWR068"
 			(at 157.48 71.12 0)
 			(effects
@@
 			(project ""
 				(path "/7933aef9-9608-4ce1-b0d8-a4ffd3b998e4/a3ca3e3d-7f11-4e5a-900e-b192a8343e04"
-					(reference "#PWR069")
+					(reference "#PWR068")
 					(unit 1)
 				)
@@
 		(dnp no)
 		(fields_autoplaced yes)
-		(property "Reference" "#PWR066"
+		(property "Reference" "#PWR065"
 			(at 134.62 119.38 0)
 			(effects
@@
 			(project ""
 				(path "/7933aef9-9608-4ce1-b0d8-a4ffd3b998e4/a3ca3e3d-7f11-4e5a-900e-b192a8343e04"
-					(reference "#PWR066")
+					(reference "#PWR065")
 					(unit 1)
 				)
@@
 		(dnp no)
 		(fields_autoplaced yes)
-		(property "Reference" "#FLG04"
+		(property "Reference" "#FLG06"
 			(at 219.71 61.595 0)
 			(effects
@@
 			(project ""
 				(path "/7933aef9-9608-4ce1-b0d8-a4ffd3b998e4/a3ca3e3d-7f11-4e5a-900e-b192a8343e04"
-					(reference "#FLG04")
+					(reference "#FLG06")
 					(unit 1)
 				)
@@
 		(dnp no)
 		(fields_autoplaced yes)
-		(property "Reference" "#PWR062"
+		(property "Reference" "#PWR061"
 			(at 45.72 114.3 0)
 			(effects
@@
 			(project ""
 				(path "/7933aef9-9608-4ce1-b0d8-a4ffd3b998e4/a3ca3e3d-7f11-4e5a-900e-b192a8343e04"
-					(reference "#PWR062")
+					(reference "#PWR061")
 					(unit 1)
 				)
@@
 		(dnp no)
 		(fields_autoplaced yes)
-		(property "Reference" "#PWR072"
+		(property "Reference" "#PWR071"
 			(at 177.8 38.1 0)
 			(effects
@@
 			(project ""
 				(path "/7933aef9-9608-4ce1-b0d8-a4ffd3b998e4/a3ca3e3d-7f11-4e5a-900e-b192a8343e04"
-					(reference "#PWR072")
+					(reference "#PWR071")
 					(unit 1)
 				)
@@
 		(dnp no)
 		(fields_autoplaced yes)
-		(property "Reference" "#FLG05"
+		(property "Reference" "#FLG07"
 			(at 219.71 79.375 0)
 			(effects
@@
 			(project ""
 				(path "/7933aef9-9608-4ce1-b0d8-a4ffd3b998e4/a3ca3e3d-7f11-4e5a-900e-b192a8343e04"
-					(reference "#FLG05")
+					(reference "#FLG07")
 					(unit 1)
 				)
@@
 		(dnp no)
 		(fields_autoplaced yes)
-		(property "Reference" "#PWR063"
+		(property "Reference" "#PWR062"
 			(at 72.39 66.04 0)
 			(effects
@@
 			(project ""
 				(path "/7933aef9-9608-4ce1-b0d8-a4ffd3b998e4/a3ca3e3d-7f11-4e5a-900e-b192a8343e04"
-					(reference "#PWR063")
+					(reference "#PWR062")
 					(unit 1)
 				)
@@
 		(dnp no)
 		(fields_autoplaced yes)
-		(property "Reference" "#PWR067"
+		(property "Reference" "#PWR066"
 			(at 146.05 50.8 0)
 			(effects
@@
 			(project ""
 				(path "/7933aef9-9608-4ce1-b0d8-a4ffd3b998e4/a3ca3e3d-7f11-4e5a-900e-b192a8343e04"
-					(reference "#PWR067")
+					(reference "#PWR066")
 					(unit 1)
 				)
@@
 		(dnp no)
 		(fields_autoplaced yes)
-		(property "Reference" "#FLG08"
+		(property "Reference" "#FLG05"
 			(at 105.41 37.465 0)
 			(effects
@@
 			(project ""
 				(path "/7933aef9-9608-4ce1-b0d8-a4ffd3b998e4/a3ca3e3d-7f11-4e5a-900e-b192a8343e04"
-					(reference "#FLG08")
+					(reference "#FLG05")
 					(unit 1)
 				)
@@
 		(dnp no)
 		(fields_autoplaced yes)
-		(property "Reference" "#PWR064"
+		(property "Reference" "#PWR063"
 			(at 83.82 66.04 0)
 			(effects
@@
 			(project ""
 				(path "/7933aef9-9608-4ce1-b0d8-a4ffd3b998e4/a3ca3e3d-7f11-4e5a-900e-b192a8343e04"
-					(reference "#PWR064")
+					(reference "#PWR063")
 					(unit 1)
 				)
@@
 		(dnp no)
 		(fields_autoplaced yes)
-		(property "Reference" "#PWR070"
+		(property "Reference" "#PWR069"
 			(at 162.56 80.01 0)
 			(effects
@@
 			(project ""
 				(path "/7933aef9-9608-4ce1-b0d8-a4ffd3b998e4/a3ca3e3d-7f11-4e5a-900e-b192a8343e04"
-					(reference "#PWR070")
+					(reference "#PWR069")
 					(unit 1)
 				)
@@
 		(dnp no)
 		(fields_autoplaced yes)
-		(property "Reference" "#PWR0104"
+		(property "Reference" "#PWR073"
 			(at 215.9 73.66 0)
 			(effects
@@
 			(project ""
 				(path "/7933aef9-9608-4ce1-b0d8-a4ffd3b998e4/a3ca3e3d-7f11-4e5a-900e-b192a8343e04"
-					(reference "#PWR0104")
+					(reference "#PWR073")
 					(unit 1)
 				)
@@
 		(on_board yes)
 		(dnp no)
-		(property "Reference" "U6"
+		(property "Reference" "U7"
 			(at 67.31 99.06 0)
 			(effects
@@
 			(project "chibarobo_board_2024"
 				(path "/7933aef9-9608-4ce1-b0d8-a4ffd3b998e4/a3ca3e3d-7f11-4e5a-900e-b192a8343e04"
-					(reference "U6")
+					(reference "U7")
 					(unit 1)
 				)
@@
 		(dnp no)
 		(fields_autoplaced yes)
-		(property "Reference" "#PWR068"
+		(property "Reference" "#PWR067"
 			(at 151.13 50.8 0)
 			(effects
@@
 			(project ""
 				(path "/7933aef9-9608-4ce1-b0d8-a4ffd3b998e4/a3ca3e3d-7f11-4e5a-900e-b192a8343e04"
-					(reference "#PWR068")
+					(reference "#PWR067")
 					(unit 1)
 				)
@@
 		(dnp no)
 		(fields_autoplaced yes)
-		(property "Reference" "R38"
+		(property "Reference" "R37"
 			(at 46.99 123.19 90)
 			(effects
@@
 			(project ""
 				(path "/7933aef9-9608-4ce1-b0d8-a4ffd3b998e4/a3ca3e3d-7f11-4e5a-900e-b192a8343e04"
-					(reference "R38")
+					(reference "R37")
 					(unit 1)
 				)
@@
 		(dnp no)
 		(fields_autoplaced yes)
-		(property "Reference" "R37"
+		(property "Reference" "R36"
 			(at 33.02 102.87 90)
 			(effects
@@
 			(project ""
 				(path "/7933aef9-9608-4ce1-b0d8-a4ffd3b998e4/a3ca3e3d-7f11-4e5a-900e-b192a8343e04"
-					(reference "R37")
+					(reference "R36")
 					(unit 1)
 				)
@@
 		(on_board yes)
 		(dnp no)
-		(property "Reference" "J16"
+		(property "Reference" "J15"
 			(at 228.6 72.3901 0)
 			(effects
@@
 			(project ""
 				(path "/7933aef9-9608-4ce1-b0d8-a4ffd3b998e4/a3ca3e3d-7f11-4e5a-900e-b192a8343e04"
-					(reference "J16")
+					(reference "J15")
 					(unit 1)
 				)
@@
 		(dnp no)
 		(fields_autoplaced yes)
-		(property "Reference" "#PWR071"
+		(property "Reference" "#PWR070"
 			(at 165.1 99.06 0)
 			(effects
@@
 			(project ""
 				(path "/7933aef9-9608-4ce1-b0d8-a4ffd3b998e4/a3ca3e3d-7f11-4e5a-900e-b192a8343e04"
-					(reference "#PWR071")
+					(reference "#PWR070")
 					(unit 1)
 				)
@@
 		(dnp no)
 		(fields_autoplaced yes)
-		(property "Reference" "U6"
+		(property "Reference" "U7"
 			(at 90.17 53.3399 0)
 			(effects
@@
 			(project "chibarobo_board_2024"
 				(path "/7933aef9-9608-4ce1-b0d8-a4ffd3b998e4/a3ca3e3d-7f11-4e5a-900e-b192a8343e04"
-					(reference "U6")
+					(reference "U7")
 					(unit 2)
 				)
@@
 		(dnp no)
 		(fields_autoplaced yes)
-		(property "Reference" "#PWR0105"
+		(property "Reference" "#PWR072"
 			(at 215.9 67.31 0)
 			(effects
@@
 			(project ""
 				(path "/7933aef9-9608-4ce1-b0d8-a4ffd3b998e4/a3ca3e3d-7f11-4e5a-900e-b192a8343e04"
-					(reference "#PWR0105")
+					(reference "#PWR072")
 					(unit 1)
 				)
@@
 		(dnp no)
 		(fields_autoplaced yes)
-		(property "Reference" "R39"
+		(property "Reference" "R38"
 			(at 88.9 100.33 90)
 			(effects
@@
 			(project ""
 				(path "/7933aef9-9608-4ce1-b0d8-a4ffd3b998e4/a3ca3e3d-7f11-4e5a-900e-b192a8343e04"
-					(reference "R39")
+					(reference "R38")
 					(unit 1)
 				)
@@
 		(dnp no)
 		(fields_autoplaced yes)
-		(property "Reference" "#PWR065"
+		(property "Reference" "#PWR064"
 			(at 105.41 50.8 0)
 			(effects
@@
 			(project ""
 				(path "/7933aef9-9608-4ce1-b0d8-a4ffd3b998e4/a3ca3e3d-7f11-4e5a-900e-b192a8343e04"
-					(reference "#PWR065")
-					(unit 1)
-				)
+					(reference "#PWR064")
+					(unit 1)
+				)

Commit message: gaber
Parts:
- D1, D3: JLCPCB Parts# (none) -> C150049
- D2: JLCPCB Parts# (none) -> C5224081
- IC3: JLCPCB Parts# (none) -> C5381644
Connections:
- net SAFE_+BATT: now also D2.1 (AR), D2.3 (AG); no longer D2.2 (K1), D2.4 (K2)
- net at D3.2 (A): now also D2.4 (CG); no longer D2.3 (A2)
- net at D1.2 (A): now also D2.2 (CR); no longer D2.1 (A1)
Changed lines of the file:
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@@
 			)
 		)
-		(property "JLCPCB Parts#" ""
+		(property "JLCPCB Parts#" "C5381644"
 			(at 134.62 107.95 0)
 			(effects
@@
 			)
 		)
-		(property "JLCPCB Parts#" ""
+		(property "JLCPCB Parts#" "C150049"
 			(at 162.56 66.04 0)
 			(effects
@@
 			)
 		)
-		(property "JLCPCB Parts#" ""
+		(property "JLCPCB Parts#" "C150049"
 			(at 157.48 66.04 0)
 			(effects
@@
 			)
 		)
-		(property "JLCPCB Parts#" ""
+		(property "JLCPCB Parts#" "C5224081"
 			(at 160.02 49.53 0)
 			(effects
