File: Servo.kicad_sch (KiCad schematic)
At the start: 30 parts, among them J1 Conn_01x03_Socket, J2 Conn_01x03_Socket, J3 Conn_01x03_Socket, J4 Conn_01x03_Socket, J5 Conn_01x03_Socket, Q3 2SA1162-GR_F_, Q4 2SA1162-GR_F_, Q5 2SA1162-GR_F_, Q6 2SA1162-GR_F_, Q7 2SA1162-GR_F_, U1 TLP291, U2 TLP291, U3 TLP291, U4 TLP291, U5 TLP291

Commit message: CircuitComplete
Parts:
- Q3, Q4, Q5, Q6, Q7: footprint SSM3K7002CFULF -> SamacSys_Parts:SSM3K7002CFULF
- renumbered J1 to J2, J2 to J3, J3 to J4, J4 to J5, J5 to J6, R13 to R12, R12 to R13
Other:
- moved on the sheet: J3, J4, J5, J6, Q4, Q5, Q6, Q7, R15, R16, R17, R18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

Commit message: Rev1
Connections:
- net +5V renamed +3.3V

Commit message: Rev1
Parts:
- Q3, Q4, Q5, Q6, Q7: footprint SamacSys_Parts:SSM3K7002CFULF -> Package_TO_SOT_SMD:SC-59; JLCPCB Parts# (none) -> C155455
- U1, U2, U3, U4, U5: JLCPCB Parts# (none) -> C5121290

Commit message: before elimination of J7
Parts:
- renumbered R12 to R11, R13 to R12, R14 to R13, R15 to R14, R16 to R15, R17 to R16, R18 to R17, R19 to R18, R20 to R19, R21 to R20, R22 to R21, R23 to R22, R24 to R23, R25 to R24, R26 to R25, U1 to U2, U2 to U3, U3 to U4, U4 to U5, U5 to U6
Connections:
- net +3.3V renamed +5V
