File: chibarobo_board_2024.kicad_pcb (KiCad board)
At the start: 2 copper layers, 142 parts, among them IC1 ESP32-S2-DevKitM-1, IC2 NCP3020ADR2G, IC3 TC74HC00AF_F_, IC4 L78M05CDT, IC5 TC7W14FK, IC6 D44H8, J1 Conn_01x18_Socket, J10 Conn_01x03_Socket, J11 Conn_01x02_Socket, J12 Conn_01x03_Socket, J13 Conn_01x03_Socket, J14 Conn_01x03_Socket, J15 Conn_01x02_Socket, J16 Conn_01x02_Socket, J2 Conn_01x03_Socket, J3 Conn_01x03_Socket, J4 Conn_01x03_Socket, J5 Conn_01x03_Socket, J6 Conn_01x03_Socket, J7 Conn_01x02_Socket, J8 Conn_01x03_Socket, J9 Conn_01x02_Socket, K1 V23134J, Q1 IRFIZ24NPbF, Q10 2SC2712-GR_TE85L,F, Q11 2SC2712-GR_TE85L,F, Q12 2SC2712-GR_TE85L,F, Q13 2SC2712-GR_TE85L,F, Q14 BUZ11, Q2 VBZM630, Q3 2SA1162-GR_F_, Q4 2SA1162-GR_F_, Q5 2SA1162-GR_F_, Q6 2SA1162-GR_F_, Q7 2SA1162-GR_F_, Q8 2SA1162-GR_F_, Q9 2SC2712-GR_TE85L,F, SW1 SW_Push, SW2 SW_Push, U1 TLP291, U2 TLP291, U3 TLP291, U4 TLP291, U5 TLP291, U6 74LVC1G123, U7 TLP291

Commit message: Rev1
Parts:
- removed IC6: D44H8, SamacSys_Parts:TO270P460X1020X2008-3P
- removed SW1, SW2: SW_Push, Button_Switch_THT:SW_PUSH_6mm_H4.3mm
- added D10: 12V_Zener, Diode_SMD:D_SOD-323, B.Cu at (142.5, 78.5)
- added Q15: NTA7002NT1G, SamacSys_Parts:SOT50P160X90-3N, F.Cu at (130.7, 94.0)
- added R62: 10k, Resistor_SMD:R_0603_1608Metric, F.Cu at (130.7, 92.2)
- added S1: SKRPACE010, SamacSys_Parts:SMT_4.2X3.2_, F.Cu at (111.5, 53.5)
- added U8: TSM3446CX6, SamacSys_Parts:SOT95P280X95-6N, B.Cu at (127.0, 91.0)
- C1, C10, C11, C13, C14, C15, C16, C17, C18, C2, C3, C4, C5, C6, C7, C8, C9, D4, D6, D7, D9, F1, IC2, IC3, IC4, IC5, Q10, Q11, Q13, Q3, Q4, Q5, Q8, Q9, R1, R12, R13, R15, R16, R18, R19, R2, R27, R29, R3, R31, R33, R35, R37, R39, R40, R41, R42, R43, R44, R45, R46, R47, R48, R49, R50, R51, R52, R53, R54, R55, R56, R59, R6, R60, R61, R7, R8, R9, U1, U2, U3, U6, U7: moved to B.Cu
- C12: footprint Capacitor_THT:CP_Radial_D5.0mm_P2.00mm -> Capacitor_SMD:C_0805_2012Metric; moved to B.Cu
- D8: footprint Diode_THT:D_5W_P10.16mm_Horizontal -> Diode_THT:D_5W_P5.08mm_Vertical_KathodeUp
- J1: value Conn_01x18_Socket -> Conn_01x14_Socket; footprint Connector_PinHeader_2.54mm:PinHeader_2x09_P2.54mm_Vertical -> Connector_PinHeader_2.54mm:PinHeader_2x07_P2.54mm_Vertical
- J15: footprint Connector_JST:JST_XH_B2B-XH-AM_1x02_P2.50mm_Vertical -> Connector_JST:JST_XH_B2B-XH-A_1x02_P2.50mm_Vertical
- L1: value PDPMAA1712-101MP -> 60B104C; footprint original:PDPMAA1712-101MP -> SamacSys_Parts:60B104C; moved to B.Cu
- Q14: value BUZ11 -> IRFL014TRPBF; footprint Package_TO_SOT_THT:TO-220-3_Vertical -> SamacSys_Parts:SOT230P700X180-4N
- Q2: value VBZM630 -> IRFR014TRPBF-BE3; footprint Package_TO_SOT_THT:TO-220-3_Vertical -> SamacSys_Parts:IRFR014TRPBFBE3; moved to B.Cu
- R57: value 510 -> 2.2k; moved to B.Cu
- R58: value 1.5 -> 1.3; footprint Resistor_SMD:R_0603_1608Metric -> Resistor_SMD:R_1206_3216Metric; moved to B.Cu
- moved J1 198.4 mm to (194.0, 61.5)
- moved H2 193.9 mm to (195.0, 55.0)
- moved IC1 193.4 mm to (166.0, 57.3)
- moved H4 189.6 mm to (195.0, 115.0)
- moved J8 165.7 mm to (195.5, 88.0)
- moved J10 165.6 mm to (195.5, 94.5)
- moved J12 165.4 mm to (195.5, 101.0)
- moved J13 165.3 mm to (195.5, 107.5)
- moved J14 156.5 mm to (185.5, 117.0), turned to 180 degrees
- moved U3 143.2 mm to (176.0, 66.0), turned to 90 degrees
- moved R16 141.9 mm to (178.5, 67.5), turned to 90 degrees
- moved U2 140.6 mm to (172.6, 61.2), turned to 90 degrees
- moved J7 140.2 mm to (165.9, 115.5)
- moved C6 139.5 mm to (142.0, 97.0), turned to -90 degrees
- moved R13 139.4 mm to (178.5, 64.5), turned to 90 degrees
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Connections:
- net /PowerSupply/MS renamed MS
- C12 pad 1: Net-(D2-K1) -> /PowerSupply/SAFE_+BATT
- D2 pad 2: Net-(D2-K1) -> /PowerSupply/SAFE_+BATT
- D2 pad 4: Net-(D2-K1) -> /PowerSupply/SAFE_+BATT
- F1 pad 1: Net-(D2-K1) -> /PowerSupply/SAFE_+BATT
- IC1 pad J328: Net-(IC1-21) -> unconnected-(IC1-21-PadJ328)
- IC1 pad J329: Net-(IC1-20) -> unconnected-(IC1-20-PadJ329)
- IC1 pad J330: Net-(IC1-19) -> unconnected-(IC1-19-PadJ330)
- IC1 pad J331: Net-(IC1-18) -> unconnected-(IC1-18-PadJ331)
- IC2 pad 4: GNDPWR -> Net-(IC2-GND)
- IC4 pad 1: Net-(D2-K1) -> /PowerSupply/SAFE_+BATT
- Q11 pad 3: Net-(IC6-B) -> Net-(D10-K)
- Q12 pad 1: Net-(IC6-E) -> Net-(Q12-BASE)
- Q12 pad 3: Net-(IC6-B) -> Net-(D10-K)
- Q2 pad 1: Net-(IC2-LSDR) -> Net-(D10-K)
- Q2 pad 2: Net-(IC2-VSW) -> GNDPWR
- Q2 pad 3: GNDPWR -> Net-(Q12-BASE)
- R13 pad 1: +5V -> +3.3V
- R16 pad 1: +5V -> +3.3V
- R19 pad 1: +5V -> +3.3V
- R22 pad 1: +5V -> +3.3V
- R25 pad 1: +5V -> +3.3V
- R57 pad 1: /PowerSupply/LOGPWR -> /PowerSupply/SAFE_+BATT
- R57 pad 2: Net-(IC6-B) -> Net-(D10-K)
- R58 pad 1: Net-(IC6-E) -> Net-(Q12-BASE)
- R60 pad 1: +BATT -> /PowerSupply/SAFE_+BATT
Routing:
- net +5V: track 0.00 -> 274.4 mm, vias 0 -> 5
- net +BATT: track 0.00 -> 262.6 mm, vias 0 -> 1
- net -BATT: track 0.00 -> 151.7 mm, vias 0 -> 3
- net ~{EMS}_{INFO}: track 0.00 -> 122.2 mm, vias 0 -> 1
- net GNDPWR: track 0.00 -> 99.7 mm, vias 0 -> 141
- net +7.5V: track 0.00 -> 96.9 mm, vias 0 -> 36
- net MS: track 0.00 -> 89.0 mm, vias 0 -> 2
- net +3.3V: track 0.00 -> 77.0 mm, vias 0 -> 3
- net Net-(J8-Pin_3): track 0.00 -> 69.1 mm
- net /PowerSupply/SAFE_+BATT: track 0.00 -> 64.8 mm, vias 0 -> 1
- net Net-(J8-Pin_2): track 0.00 -> 60.8 mm
- net Net-(J10-Pin_3): track 0.00 -> 60.7 mm
- net Net-(J10-Pin_2): track 0.00 -> 52.3 mm
- net Net-(J12-Pin_3): track 0.00 -> 52.2 mm
- net Net-(D8-A): track 0.00 -> 51.1 mm, vias 0 -> 1
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- added copper zone on B.Cu, net +7.5V
- added copper zone on F.Cu, net +7.5V
- added copper zone on B.Cu, net GND
- added copper zone on F.Cu, net GND
- added copper zone on B.Cu, net GNDPWR
- added copper zone on F.Cu, net GNDPWR
Other:
- board outline added: 100 x 70 mm
- board text added: "26"
- board text added: "33"
- board text added: "34"
- board text added: "35"
- board text added: "36"
- board text added: "37"
- board text added: "38"
- board text added: "39"
- board text added: "3V3"
- board text added: "40"
- board text added: "41"
- board text added: "5V"
- board text added: "ChibaRoboBoard 2024"
- board text added: "DIR"
- board text added: "G"
- board text added: "GND"
- board text added: "OVERRIDE"
- board text added: "PWM"
- board text added: "Rev1"
- board text added: "VCC"
- board text added: "~{EMS}"

Commit message: Rev1
Parts:
- D4: footprint Diode_SMD:D_SOD-323 -> Diode_SMD:D_SOD-323F
- Q3, Q4, Q5, Q6, Q7, Q8: footprint SamacSys_Parts:SSM3K7002CFULF -> Package_TO_SOT_SMD:SC-59
- moved R24 0.49 mm to (169.8, 70.9)
- moved Q7 0.32 mm to (170.2, 68.3), turned to 180 degrees
- moved R43 0.29 mm to (111.8, 59.2)
- moved R21 0.17 mm to (169.8, 65.8)
- moved R47 0.14 mm to (114.5, 59.2)
- turned Q6 to 180 degrees
- turned Q4 to 90 degrees
- turned Q3 to 90 degrees
- turned Q5 to 90 degrees
- turned Q8 to 180 degrees
Routing:
- net Net-(Q5-Pad1): track 4.80 -> 5.46 mm
- net Net-(Q10-COLLECTOR): track 17.6 -> 17.0 mm
- net Net-(Q8-Pad1): track 1.95 -> 2.46 mm
- net /Servo/Servo1: track 5.31 -> 5.82 mm
- net GND: vias 86 -> 87

Commit message: Rev1.1
Parts:
- R44: value 62 -> 100
- moved S1 0.51 mm to (112.0, 53.6), turned to -90 degrees
Connections:
- S1 pad 1: GND -> Net-(IC5-1A)
- S1 pad 2: Net-(IC5-1A) -> unconnected-(S1-Pad2)
- S1 pad 4: Net-(IC5-1A) -> unconnected-(S1-Pad4)
Routing:
- net GND: track 32.4 -> 29.9 mm
- net Net-(IC5-1A): track 28.2 -> 25.7 mm
Other:
- board text added: "Rev1.1"
- board text removed: "Rev1"

Commit message: before elimination of J7
Parts:
- removed the R10 at (129.0, 101.0)
- removed the R11 at (129.0, 98.0)
- C2: value 33p -> 18p
- C3: value 1n -> 3.3n
- C4, C5: moved to F.Cu
- HS1: value Heatsink -> BPUE56-25; footprint original:BPUG56 -> original:BPUE56
- L1: footprint SamacSys_Parts:60B104C -> original:60B104C_correct
- R2: value 48 -> 18
- R3: value 220 -> 1.6k
- R4: value 2.2k -> 13k
- R5: value 330 -> 4.7k
- R6: value 16k -> 3k
- R7: value 16k -> 56k
- R9: value 27k -> 56k
- moved D1 18.8 mm to (102.0, 98.8)
- moved D2 18.8 mm to (102.0, 82.8)
- moved D3 18.8 mm to (102.0, 93.8)
- moved L1 3.50 mm to (109.5, 96.0)
- moved R58 2.55 mm to (143.0, 61.5), turned to -90 degrees
- moved R6 2.51 mm to (140.5, 97.3)
- moved R7 2.51 mm to (140.5, 100.5)
- moved C10 1.72 mm to (133.0, 67.5), turned to 90 degrees
- moved C6 1.12 mm to (143.0, 97.5)
- moved C2 0.98 mm to (138.5, 97.3)
- moved C3 0.98 mm to (138.5, 100.5)
- moved F1 0.50 mm to (144.0, 68.5)
- moved R59 0.50 mm to (144.0, 66.0)
- moved IC4 0.21 mm to (138.2, 62.1)
- renumbered D8 to D10, D10 to D8, J16 to J15, J15 to J16, Q15 to Q1, Q2 to Q12, Q12 to Q13, Q13 to Q14, Q14 to Q15, Q1 to Q2, R8 to R10, R12 to R11, R13 to R12, R14 to R13, R15 to R14, R16 to R15, R17 to R16, R18 to R17, R19 to R18, R20 to R19, R21 to R20, R22 to R21, R23 to R22, R24 to R23, R25 to R24, R26 to R25, R27 to R26, R28 to R27, R29 to R28, R30 to R29, R31 to R30, R32 to R31, R33 to R32, R34 to R33, R35 to R34, R36 to R35, R37 to R36, R38 to R37, R39 to R38, R40 to R39, R41 to R40, R42 to R41, R43 to R42, R44 to R43, R45 to R44, R46 to R45, R47 to R46, R48 to R47, R49 to R48, R50 to R49, R51 to R50, R52 to R51, R53 to R52, R54 to R53, R55 to R54, R56 to R55, R57 to R56, R58 to R57, R59 to R58, R60 to R59, R61 to R60, R62 to R8, U8 to U1, U1 to U2, U2 to U3, U3 to U4, U4 to U5, U5 to U6, U6 to U7, U7 to U8
Connections:
- C2 pad 1: /ActuatorPowerSupply/FB -> GNDPWR
- IC4 pad 2: /PowerSupply/LOGPWR -> -BATT
- IC4 pad 3: -BATT -> /PowerSupply/LOGPWR
- R12 pad 1: +3.3V -> +5V
- R15 pad 1: +3.3V -> +5V
- R18 pad 1: +3.3V -> +5V
- R21 pad 1: +3.3V -> +5V
- R24 pad 1: +3.3V -> +5V
- R6 pad 1: /ActuatorPowerSupply/FB -> GNDPWR
Routing:
- net +3.3V: track 77.0 -> 51.7 mm, vias 3 -> 1
- net -BATT: track 151.7 -> 176.6 mm
- net /PowerSupply/SAFE_+BATT: track 64.8 -> 80.3 mm
- net /PowerSupply/LOGPWR: track 44.0 -> 58.8 mm
- net +5V: track 274.4 -> 284.3 mm, vias 5 -> 7
- net /ActuatorPowerSupply/FB: track 20.1 -> 11.1 mm
- net Net-(IC2-VSW): track 42.9 -> 46.4 mm
- net /ActuatorPowerSupply/COMP: track 9.47 -> 6.19 mm
- net Net-(Q14-BASE): track 22.3 -> 25.3 mm
- net +7.5V: track 96.9 -> 93.9 mm
- net GNDPWR: track 99.7 -> 98.0 mm, vias 141 -> 143
- net Net-(D2-A2): track 13.7 -> 12.1 mm
- net +BATT: track 262.6 -> 264.0 mm
- net Net-(Q14-COLLECTOR): track 23.6 -> 22.8 mm
- net ~{EMS}_{INFO}: track 122.2 -> 122.9 mm
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
Commit message: Rev1.2
Parts:
- removed the J7 at (165.9, 115.5)
- renumbered J11 to J10, J12 to J11, J13 to J12, J14 to J13, J15 to J14, J16 to J15, J8 to J7, J9 to J8, J10 to J9
Routing:
- net GNDPWR: track 98.0 -> 78.0 mm
- net +BATT: track 264.0 -> 245.3 mm
- net +5V: track 284.3 -> 276.0 mm
Other:
- board text added: "Rev1.2"
- board text removed: "Rev1.1"
