File: chibarobo_board_2024.kicad_pcb (KiCad board)
At the start: 2 copper layers, 100 x 70 mm, 142 parts, among them IC1 ESP32-S2-DevKitM-1, IC2 NCP3020ADR2G, IC3 TC74HC00AF_F_, IC4 L78M05CDT, IC5 TC7W14FK, J1 Conn_01x14_Socket, J10 Conn_01x03_Socket, J11 Conn_01x02_Socket, J12 Conn_01x03_Socket, J13 Conn_01x03_Socket, J14 Conn_01x03_Socket, J15 Conn_01x02_Socket, J16 Conn_01x02_Socket, J2 Conn_01x03_Socket, J3 Conn_01x03_Socket, J4 Conn_01x03_Socket, J5 Conn_01x03_Socket, J6 Conn_01x03_Socket, J7 Conn_01x02_Socket, J8 Conn_01x03_Socket, J9 Conn_01x02_Socket, K1 V23134J, Q1 NTA7002NT1G, Q10 2SC2712-GR_TE85L,F, Q11 2SC2712-GR_TE85L,F, Q12 IRFR014TRPBF-BE3, Q13 2SC2712-GR_TE85L,F, Q14 2SC2712-GR_TE85L,F, Q15 IRFL014TRPBF, Q2 IRFIZ24NPbF, Q3 2SA1162-GR_F_, Q4 2SA1162-GR_F_, Q5 2SA1162-GR_F_, Q6 2SA1162-GR_F_, Q7 2SA1162-GR_F_, Q8 2SA1162-GR_F_, Q9 2SC2712-GR_TE85L,F, U1 TSM3446CX6, U2 TLP291, U3 TLP291, U4 TLP291, U5 TLP291, U6 TLP291, U7 74LVC1G123, U8 TLP291

Commit message: Rev1.2
Parts:
- Q4, Q5, R14, R15, R17, R18, R26, R28, R30, R32, R34, U3, U4: moved to F.Cu
- Q6, Q7, R13, R20, R21, R23, R24, R27, R29, R31, R33, R35: moved to B.Cu
- moved J1 47.1 mm to (197.0, 108.5), turned to 180 degrees
- moved J14 31.1 mm to (195.5, 87.5), turned to 0 degrees
- moved J10 26.5 mm to (195.5, 68.0)
- moved J12 26.5 mm to (195.5, 74.5)
- moved J13 26.5 mm to (195.5, 81.0)
- moved J8 26.5 mm to (195.5, 61.5)
- moved R27 21.5 mm to (168.0, 66.5)
- moved R29 21.5 mm to (168.0, 69.5)
- moved R31 21.5 mm to (168.0, 72.5)
- moved R33 21.5 mm to (168.0, 75.5)
- moved R35 21.5 mm to (168.0, 78.5)
- moved R11 11.1 mm to (173.0, 56.5)
- moved R13 7.18 mm to (164.0, 54.5), turned to 90 degrees
- moved R15 6.18 mm to (177.0, 61.5)
- moved R18 6.18 mm to (177.0, 64.5)
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Connections:
- IC1 pad J123: /Servo/Servo1 -> unconnected-(IC1-11-PadJ123)
- IC1 pad J124: /Servo/Servo2 -> unconnected-(IC1-12-PadJ124)
- IC1 pad J125: /Servo/Servo3 -> unconnected-(IC1-13-PadJ125)
- IC1 pad J126: /Servo/Servo4 -> unconnected-(IC1-14-PadJ126)
- IC1 pad J127: /Servo/Servo5 -> unconnected-(IC1-15-PadJ127)
- IC1 pad J327: unconnected-(IC1-26-PadJ327) -> /Servo/Servo5
- IC1 pad J328: unconnected-(IC1-21-PadJ328) -> /Servo/Servo4
- IC1 pad J329: unconnected-(IC1-20-PadJ329) -> /Servo/Servo3
- IC1 pad J330: unconnected-(IC1-19-PadJ330) -> /Servo/Servo2
- IC1 pad J331: unconnected-(IC1-18-PadJ331) -> /Servo/Servo1
Routing:
- net (no net): track 56.9 -> 0.00 mm
- net +5V: track 251.2 -> 293.8 mm, vias 7 -> 5
- net Net-(IC1-9): track 3.35 -> 23.0 mm
- net Net-(J14-Pin_3): track 37.0 -> 56.0 mm
- net +3.3V: track 28.7 -> 9.84 mm, vias 1 -> 0
- net Net-(IC1-5): track 0.00 -> 17.1 mm
- net Net-(IC1-7): track 4.48 -> 19.5 mm
- net Net-(IC1-10): track 5.65 -> 20.4 mm
- net Net-(J8-Pin_2): track 60.8 -> 46.2 mm
- net Net-(J14-Pin_2): track 24.2 -> 38.6 mm
- net Net-(IC1-3): track 0.00 -> 13.9 mm
- net Net-(Q6-Pad3): track 0.76 -> 13.2 mm, vias 0 -> 1
- net Net-(IC1-4): track 0.00 -> 12.0 mm
- net Net-(J10-Pin_2): track 52.3 -> 40.8 mm
- net Net-(J13-Pin_3): track 43.8 -> 55.2 mm
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Other:
- board text added: "0"
- board text added: "1"
- board text added: "10"
- board text added: "2"
- board text added: "3"
- board text added: "4"
- board text added: "5"
- board text added: "6"
- board text added: "7"
- board text added: "8"
- board text added: "9"
- board text added: "Rev2"
- board text removed: "26"
- board text removed: "33"
- board text removed: "34"
- board text removed: "35"
- board text removed: "36"
- board text removed: "37"
- board text removed: "38"
- board text removed: "39"
- board text removed: "40"
- board text removed: "41"
- board text removed: "Rev1.1"
- board text removed: "~{EMS}"
