File: chibarobo_board_2024.kicad_pcb (KiCad board)
At the start: 2 copper layers, 100 x 70 mm, 142 parts, among them IC1 ESP32-S2-DevKitM-1, IC2 NCP3020ADR2G, IC3 TC74HC00AF_F_, IC4 L78M05CDT, IC5 TC7W14FK, J1 Conn_01x14_Socket, J10 Conn_01x03_Socket, J11 Conn_01x02_Socket, J12 Conn_01x03_Socket, J13 Conn_01x03_Socket, J14 Conn_01x03_Socket, J15 Conn_01x02_Socket, J16 Conn_01x02_Socket, J2 Conn_01x03_Socket, J3 Conn_01x03_Socket, J4 Conn_01x03_Socket, J5 Conn_01x03_Socket, J6 Conn_01x03_Socket, J7 Conn_01x02_Socket, J8 Conn_01x03_Socket, J9 Conn_01x02_Socket, K1 V23134J, Q1 NTA7002NT1G, Q10 2SC2712-GR_TE85L,F, Q11 2SC2712-GR_TE85L,F, Q12 IRFR014TRPBF-BE3, Q13 2SC2712-GR_TE85L,F, Q14 2SC2712-GR_TE85L,F, Q15 IRFL014TRPBF, Q2 IRFIZ24NPbF, Q3 2SA1162-GR_F_, Q4 2SA1162-GR_F_, Q5 2SA1162-GR_F_, Q6 2SA1162-GR_F_, Q7 2SA1162-GR_F_, Q8 2SA1162-GR_F_, Q9 2SC2712-GR_TE85L,F, U1 TSM3446CX6, U2 TLP291, U3 TLP291, U4 TLP291, U5 TLP291, U6 TLP291, U7 74LVC1G123, U8 TLP291

Commit message: gaber
Parts:
- moved D1 5.20 mm to (102.0, 93.7)
- moved D3 4.50 mm to (102.0, 98.3)
- turned D2 to -90 degrees
Connections:
- D2 pad 1: Net-(D1-A) -> /PowerSupply/SAFE_+BATT
- D2 pad 2: /PowerSupply/SAFE_+BATT -> Net-(D1-A)
- D2 pad 3: Net-(D2-A2) -> /PowerSupply/SAFE_+BATT
- D2 pad 4: /PowerSupply/SAFE_+BATT -> Net-(D2-CG)
- D3 pad 2: Net-(D2-A2) -> Net-(D2-CG)
Routing:
- net Net-(D2-CG): track 0.00 -> 16.4 mm
- net Net-(D2-A2): track 12.1 -> 0.00 mm
- net Net-(D1-A): track 13.9 -> 8.36 mm
- net -BATT: track 176.6 -> 171.4 mm
- net /PowerSupply/SAFE_+BATT: track 80.3 -> 81.4 mm
Changed lines of the file:
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@@
 	(net 20 "Net-(D9-K)")
 	(net 21 "Net-(D1-A)")
-	(net 22 "Net-(D2-A2)")
+	(net 22 "Net-(D2-CG)")
 	(net 23 "Net-(D4-K)")
 	(net 24 "/PowerSupply/EMS/OVERRIDE")
@@
 	(footprint "Diode_SMD:D_SOD-123"
 		(layer "F.Cu")
-		(at 102 93.85 90)
+		(at 102 98.35 90)
 		(descr "SOD-123")
 		(tags "SOD-123")
@@
 			(layers "F.Cu" "F.Paste" "F.Mask")
 			(roundrect_rratio 0.25)
-			(net 22 "Net-(D2-A2)")
+			(net 22 "Net-(D2-CG)")
 			(pinfunction "A")
 			(pintype "passive")
@@
 		(fp_arc
 			(start 16 -2.2)
-			(mid 15.263943 0.453213)
+			(mid 15.263944 0.453214)
 			(end 13.316806 2.4)
 			(stroke
@@
 	(footprint "LED_SMD:LED_Avago_PLCC4_3.2x2.8mm_CW"
 		(layer "F.Cu")
-		(at 102 82.85 90)
+		(at 102 82.85 -90)
 		(descr "3.2mm x 2.8mm PLCC4 RGB LED, https://docs.broadcom.com/docs/AV02-4186EN")
 		(tags "LED Avago PLCC-4 3528 ASMB-MTB0-0A3A2")
@@
 		)
 		(property "Footprint" "LED_SMD:LED_Avago_PLCC4_3.2x2.8mm_CW"
-			(at 0 0 90)
+			(at 0 0 -90)
 			(unlocked yes)
 			(layer "F.Fab")
@@
 		)
 		(property "Datasheet" "https://www.vishay.com/docs/81359/vlmkg34.pdf"
-			(at 0 0 90)
+			(at 0 0 -90)
 			(unlocked yes)
 			(layer "F.Fab")
@@
 		)
 		(property "Description" "Dual LED, cathodes on pins 1 and 3"
-			(at 0 0 90)
+			(at 0 0 -90)
 			(unlocked yes)
 			(layer "F.Fab")
@@
 		)
 		(property "JLCPCB Parts#" ""
-			(at 0 0 90)
+			(at 0 0 -90)
 			(unlocked yes)
 			(layer "F.Fab")
@@
 		(attr smd)
 		(fp_line
-			(start -2.500044 -1.5)
-			(end 1.95 -1.5)
+			(start -1.95 1.5)
+			(end 1.95 1.5)
 			(stroke
 				(width 0.12)
@@
 		)
 		(fp_line
-			(start -1.95 1.5)
-			(end 1.95 1.5)
+			(start -2.500044 -1.5)
+			(end 1.95 -1.5)
 			(stroke
 				(width 0.12)
@@
 		)
 		(fp_line
-			(start -2.5 -1.65)
-			(end 2.5 -1.65)
+			(start 2.5 1.65)
+			(end -2.5 1.65)
 			(stroke
 				(width 0.05)
@@
 		)
 		(fp_line
-			(start -2.5 -1.65)
-			(end -2.5 1.65)
+			(start 2.5 1.65)
+			(end 2.5 -1.65)
 			(stroke
 				(width 0.05)
@@
 		)
 		(fp_line
-			(start 2.5 1.65)
-			(end 2.5 -1.65)
+			(start -2.5 -1.65)
+			(end -2.5 1.65)
 			(stroke
 				(width 0.05)
@@
 		)
 		(fp_line
-			(start 2.5 1.65)
-			(end -2.5 1.65)
+			(start -2.5 -1.65)
+			(end 2.5 -1.65)
 			(stroke
 				(width 0.05)
@@
 		)
 		(fp_line
-			(start 1.6 -1.4)
-			(end -1.6 -1.4)
+			(start -1.6 1.4)
+			(end 1.6 1.4)
 			(stroke
 				(width 0.1)
@@
 		)
 		(fp_line
-			(start -0.6 -1.4)
-			(end -1.6 -0.4)
+			(start 1.6 1.4)
+			(end 1.6 -1.4)
 			(stroke
 				(width 0.1)
@@
 		)
 		(fp_line
-			(start 1.6 1.4)
-			(end 1.6 -1.4)
+			(start -0.6 -1.4)
+			(end -1.6 -0.4)
 			(stroke
 				(width 0.1)
@@
 		)
 		(fp_line
-			(start -1.6 1.4)
-			(end 1.6 1.4)
+			(start 1.6 -1.4)
+			(end -1.6 -1.4)
 			(stroke
 				(width 0.1)
@@
 		)
 		(pad "1" smd rect
-			(at -1.5 -0.75 90)
+			(at -1.5 -0.75 270)
 			(size 1.5 1.1)
 			(layers "F.Cu" "F.Paste" "F.Mask")
-			(net 21 "Net-(D1-A)")
-			(pinfunction "A1")
+			(net 13 "/PowerSupply/SAFE_+BATT")
+			(pinfunction "AR")
 			(pintype "input")
 		)
 		(pad "2" smd rect
-			(at 1.5 -0.75 90)
+			(at 1.5 -0.75 270)
 			(size 1.5 1.1)
 			(layers "F.Cu" "F.Paste" "F.Mask")
-			(net 13 "/PowerSupply/SAFE_+BATT")
-			(pinfunction "K1")
+			(net 21 "Net-(D1-A)")
+			(pinfunction "CR")
 			(pintype "input")
 		)
 		(pad "3" smd rect
-			(at 1.5 0.75 90)
+			(at 1.5 0.75 270)
 			(size 1.5 1.1)
 			(layers "F.Cu" "F.Paste" "F.Mask")
-			(net 22 "Net-(D2-A2)")
-			(pinfunction "A2")
+			(net 13 "/PowerSupply/SAFE_+BATT")
+			(pinfunction "AG")
 			(pintype "input")
 		)
 		(pad "4" smd rect
-			(at -1.5 0.75 90)
+			(at -1.5 0.75 270)
 			(size 1.5 1.1)
 			(layers "F.Cu" "F.Paste" "F.Mask")
-			(net 13 "/PowerSupply/SAFE_+BATT")
-			(pinfunction "K2")
+			(net 22 "Net-(D2-CG)")
+			(pinfunction "CG")
 			(pintype "input")
 		)
@@
 	(footprint "Diode_SMD:D_SOD-123"
 		(layer "F.Cu")
-		(at 102 98.85 90)
+		(at 102 93.65 90)
 		(descr "SOD-123")
 		(tags "SOD-123")
@@
 	)
 	(segment
-		(start 103.5 97.048696)
-		(end 102 98.548696)
-		(width 0.2)
-		(layer "F.Cu")
-		(net 10)
-	)
-	(segment
-		(start 103.5 87)
-		(end 103.5 97.048696)
+		(start 103.5 93.8)
+		(end 102 95.3)
 		(width 0.2)
 		(layer "F.Cu")
@@
 	)
 	(segment
-		(start 148 80.5)
-		(end 150.5 83)
-		(width 0.5)
+		(start 103.5 87)
+		(end 103.5 93.8)
+		(width 0.2)
 		(layer "F.Cu")
 		(net 10)
 	)
 	(segment
-		(start 102 98.548696)
-		(end 102 100.5)
-		(width 0.2)
+		(start 148 80.5)
+		(end 150.5 83)
+		(width 0.5)
 		(layer "F.Cu")
 		(net 10)
@@
 	)
 	(segment
-		(start 103.3 59.5)
-		(end 101.25 61.55)
+		(start 133.5 59.5)
+		(end 103.3 59.5)
 		(width 0.2)
 		(layer "F.Cu")
@@
 	)
 	(segment
-		(start 133.5 59.5)
-		(end 103.3 59.5)
+		(start 102.75 81.35)
+		(end 102.5 81.6)
 		(width 0.2)
 		(layer "F.Cu")
@@
 	)
 	(segment
-		(start 133.5 59.5)
-		(end 141 67)
+		(start 102.75 80.4)
+		(end 102.75 81.35)
 		(width 0.2)
 		(layer "F.Cu")
@@
 	)
 	(segment
-		(start 101.25 81.35)
-		(end 101.25 82.45)
+		(start 102.5 82.15)
+		(end 101.25 83.4)
 		(width 0.2)
 		(layer "F.Cu")
@@
 	)
 	(segment
-		(start 101.25 82.45)
-		(end 102.75 83.95)
+		(start 101.25 83.4)
+		(end 101.25 84.35)
 		(width 0.2)
 		(layer "F.Cu")
@@
 	(segment
 		(start 101.25 61.55)
-		(end 101.25 81.35)
+		(end 101.25 79.75)
 		(width 0.2)
 		(layer "F.Cu")
@@
 	)
 	(segment
-		(start 102.75 83.95)
-		(end 102.75 84.35)
+		(start 103.3 59.5)
+		(end 101.25 61.55)
+		(width 0.2)
+		(layer "F.Cu")
+		(net 13)
+	)
+	(segment
+		(start 102.65 80.3)
+		(end 102.75 80.4)
+		(width 0.2)
+		(layer "F.Cu")
+		(net 13)
+	)
+	(segment
+		(start 102.5 81.6)
+		(end 102.5 82.15)
+		(width 0.2)
+		(layer "F.Cu")
+		(net 13)
+	)
+	(segment
+		(start 101.25 79.75)
+		(end 101.8 80.3)
+		(width 0.2)
+		(layer "F.Cu")
+		(net 13)
+	)
+	(segment
+		(start 141 67)
+		(end 133.5 59.5)
+		(width 0.2)
+		(layer "F.Cu")
+		(net 13)
+	)
+	(segment
+		(start 101.8 80.3)
+		(end 102.65 80.3)
 		(width 0.2)
 		(layer "F.Cu")
@@
 	)
 	(segment
-		(start 100.4 85.2)
-		(end 100.4 95.6)
+		(start 102.75 83.95)
+		(end 102.75 84.35)
 		(width 0.2)
 		(layer "F.Cu")
@@
 	)
 	(segment
-		(start 101.25 84.35)
-		(end 100.4 85.2)
+		(start 102 87)
+		(end 102.75 86.25)
 		(width 0.2)
 		(layer "F.Cu")
@@
 	)
 	(segment
-		(start 100.4 95.6)
-		(end 102 97.2)
+		(start 102 92)
+		(end 102 87)
 		(width 0.2)
 		(layer "F.Cu")
@@
 	)
 	(segment
-		(start 102.5 81.6)
-		(end 103.6 82.7)
-		(width 0.2)
-		(layer "F.Cu")
-		(net 22)
-	)
-	(segment
-		(start 102.75 81.35)
-		(end 102.5 81.6)
+		(start 102.75 86.25)
+		(end 102.75 84.35)
 		(width 0.2)
 		(layer "F.Cu")
-		(net 22)
+		(net 21)
 	)
 	(segment
-		(start 102 87)
-		(end 102 92.2)
+		(start 100.4 95.1)
+		(end 100.4 82.2)
 		(width 0.2)
 		(layer "F.Cu")
@@
 	)
 	(segment
-		(start 103.6 82.7)
-		(end 103.6 85.4)
+		(start 102 96.7)
+		(end 100.4 95.1)
 		(width 0.2)
 		(layer "F.Cu")
@@
 	)
 	(segment
-		(start 103.6 85.4)
-		(end 102 87)
+		(start 100.4 82.2)
+		(end 101.25 81.35)
 		(width 0.2)
 		(layer "F.Cu")
