File: chibarobo_board_2024.kicad_sch (KiCad schematic)
At the start: 0 parts

Commit message: CircuitComplete
Parts:
- added H1, H2, H3, H4: MountingHole, MountingHole:MountingHole_3.2mm_M3, symbol Mechanical:MountingHole
- added IC1: ESP32-S2-DevKitM-1, original:ESP32S2DevKitM1, symbol SamacSys_Parts:ESP32-S2-DevKitM-1
- added J1: Conn_01x18_Socket, Connector_PinHeader_2.54mm:PinHeader_2x09_P2.54mm_Vertical, symbol Connector:Conn_01x18_Socket
Connections:
- new net: IC1.J318 (41), J1.5 (Pin_5)
- new net: IC1.J319 (40), J1.6 (Pin_6)
- new net: IC1.J320 (39), J1.7 (Pin_7)
- new net: IC1.J321 (38), J1.8 (Pin_8)
- new net: IC1.J322 (37), J1.9 (Pin_9)
- new net: IC1.J323 (36), J1.10 (Pin_10)
- new net: IC1.J324 (35), J1.11 (Pin_11)
- new net: IC1.J325 (34), J1.12 (Pin_12)
- new net: IC1.J326 (33), J1.13 (Pin_13)
- new net: IC1.J327 (26), J1.14 (Pin_14)
- new net: IC1.J328 (21), J1.15 (Pin_15)
- new net: IC1.J329 (20), J1.16 (Pin_16)
- new net: IC1.J330 (19), J1.17 (Pin_17)
- new net: IC1.J331 (18), J1.18 (Pin_18)
- new net +3.3V: IC1.J111 (3V3), J1.3 (Pin_3)
- new net +5V: IC1.J130 (5V), J1.2 (Pin_2)
- new net DCMotor/DIR1: IC1.J118 (6)
- new net DCMotor/DIR2: IC1.J119 (7)
- new net DCMotor/DIR3: IC1.J120 (8)
- new net DCMotor/DIR4: IC1.J121 (9)
- new net DCMotor/DIR5: IC1.J122 (10)
- new net DCMotor/PWM1: IC1.J123 (11)
- new net DCMotor/PWM2: IC1.J124 (12)
- new net DCMotor/PWM3: IC1.J125 (13)
- new net DCMotor/PWM4: IC1.J126 (14)
- new net DCMotor/PWM5: IC1.J127 (15)
- new net GND: IC1.J131 (G_1), IC1.J311 (G_2), J1.1 (Pin_1)
- new net Servo/Servo1: IC1.J113 (1)
- new net Servo/Servo2: IC1.J114 (2)
- new net Servo/Servo3: IC1.J115 (3)
- new net Servo/Servo4: IC1.J116 (4)
- new net Servo/Servo5: IC1.J117 (5)
- new net ~{EMS}_{INFO}: IC1.J317 (42), J1.4 (Pin_4)
- no-connect marks 0 -> 8
Other:
- sheet DCMotor ports: added DIR1, DIR2, DIR3, DIR4, DIR5, PWM1, PWM2, PWM3, PWM4, PWM5; removed none
- sheet Servo ports: added Servo1, Servo2, Servo3, Servo4, Servo5; removed none

Commit message: Rev1
Parts:
- removed J1: Conn_01x18_Socket, Connector_PinHeader_2.54mm:PinHeader_2x09_P2.54mm_Vertical, symbol Connector:Conn_01x18_Socket
- added J1: Conn_01x14_Socket, Connector_PinHeader_2.54mm:PinHeader_2x07_P2.54mm_Vertical, symbol Connector:Conn_01x14_Socket
Connections:
- net +3.3V: now also J1.3 (Pin_3)
- net +5V: now also J1.2 (Pin_2)
- net GND: now also J1.1 (Pin_1)
- net ~{EMS}_{INFO}: now also J1.4 (Pin_4)
- net at IC1.J318 (41): now also J1.5 (Pin_5)
- net at IC1.J319 (40): now also J1.6 (Pin_6)
- net at IC1.J320 (39): now also J1.7 (Pin_7)
- net at IC1.J321 (38): now also J1.8 (Pin_8)
- net at IC1.J322 (37): now also J1.9 (Pin_9)
- net at IC1.J323 (36): now also J1.10 (Pin_10)
- net at IC1.J324 (35): now also J1.11 (Pin_11)
- net at IC1.J325 (34): now also J1.12 (Pin_12)
- net at IC1.J326 (33): now also J1.13 (Pin_13)
- net at IC1.J327 (26): now also J1.14 (Pin_14)
- no-connect marks 8 -> 12
Changed lines of the file:
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@@
+	)
+	(no_connect
+		(at 171.45 114.3)
 	)
 	(no_connect
@@
 	)
 	(no_connect
+		(at 171.45 109.22)
+	)
+	(no_connect
 		(at 171.45 73.66)
+	)
+	(no_connect
+		(at 171.45 111.76)
 	)
 	(no_connect
@@
 	)
 	(no_connect
+		(at 171.45 106.68)
+	)
+	(no_connect
 		(at 146.05 66.04)
 	)
@@
 	(wire
 		(pts
-			(xy 171.45 106.68) (xy 196.85 106.68)
-		)
-		(stroke
-			(width 0)
-			(type default)
-		)
-	)
-	(wire
-		(pts
 			(xy 171.45 91.44) (xy 196.85 91.44)
 		)
@@
 	(wire
 		(pts
-			(xy 171.45 111.76) (xy 196.85 111.76)
-		)
-		(stroke
-			(width 0)
-			(type default)
-		)
-	)
-	(wire
-		(pts
 			(xy 171.45 93.98) (xy 196.85 93.98)
 		)
@@
 	(wire
 		(pts
-			(xy 171.45 109.22) (xy 196.85 109.22)
-		)
-		(stroke
-			(width 0)
-			(type default)
-		)
-	)
-	(wire
-		(pts
 			(xy 115.57 110.49) (xy 115.57 121.92)
 		)
@@
 		(pts
 			(xy 123.19 88.9) (xy 146.05 88.9)
-		)
-		(stroke
-			(width 0)
-			(type default)
-		)
-	)
-	(wire
-		(pts
-			(xy 171.45 114.3) (xy 196.85 114.3)
 		)
 		(stroke
@@
 	)
 	(symbol
-		(lib_id "Connector:Conn_01x18_Socket")
-		(at 201.93 91.44 0)
+		(lib_id "Connector:Conn_01x14_Socket")
+		(at 201.93 86.36 0)
 		(unit 1)
 		(exclude_from_sim no)
@@
 		(fields_autoplaced yes)
 		(property "Reference" "J1"
-			(at 203.2 91.4399 0)
-			(effects
-				(font
-					(size 1.27 1.27)
-				)
-				(justify left)
-			)
-		)
-		(property "Value" "Conn_01x18_Socket"
-			(at 203.2 93.9799 0)
-			(effects
-				(font
-					(size 1.27 1.27)
-				)
-				(justify left)
-			)
-		)
-		(property "Footprint" "Connector_PinHeader_2.54mm:PinHeader_2x09_P2.54mm_Vertical"
-			(at 201.93 91.44 0)
+			(at 203.2 86.3599 0)
+			(effects
+				(font
+					(size 1.27 1.27)
+				)
+				(justify left)
+			)
+		)
+		(property "Value" "Conn_01x14_Socket"
+			(at 203.2 88.8999 0)
+			(effects
+				(font
+					(size 1.27 1.27)
+				)
+				(justify left)
+			)
+		)
+		(property "Footprint" "Connector_PinHeader_2.54mm:PinHeader_2x07_P2.54mm_Vertical"
+			(at 201.93 86.36 0)
 			(effects
 				(font
@@
 		)
 		(property "Datasheet" "~"
-			(at 201.93 91.44 0)
-			(effects
-				(font
-					(size 1.27 1.27)
-				)
-				(hide yes)
-			)
-		)
-		(property "Description" "Generic connector, single row, 01x18, script generated"
-			(at 201.93 91.44 0)
-			(effects
-				(font
-					(size 1.27 1.27)
-				)
-				(hide yes)
-			)
+			(at 201.93 86.36 0)
+			(effects
+				(font
+					(size 1.27 1.27)
+				)
+				(hide yes)
+			)
+		)
+		(property "Description" "Generic connector, single row, 01x14, script generated"
+			(at 201.93 86.36 0)
+			(effects
+				(font
+					(size 1.27 1.27)
+				)
+				(hide yes)
+			)
+		)
+		(pin "12"
+		)
+		(pin "9"
+		)
+		(pin "11"
+		)
+		(pin "3"
+		)
+		(pin "10"
+		)
+		(pin "6"
+		)
+		(pin "7"
 		)
 		(pin "1"
 		)
+		(pin "13"
+		)
+		(pin "8"
+		)
+		(pin "4"
+		)
+		(pin "2"
+		)
+		(pin "14"
+		)
 		(pin "5"
 		)
-		(pin "15"
-		)
-		(pin "18"
-		)
-		(pin "16"
-		)
-		(pin "3"
-		)
-		(pin "11"
-		)
-		(pin "6"
-		)
-		(pin "10"
-		)
-		(pin "14"
-		)
-		(pin "12"
-		)
-		(pin "8"
-		)
-		(pin "2"
-		)
-		(pin "7"
-		)
-		(pin "4"
-		)
-		(pin "17"
-		)
-		(pin "9"
-		)
-		(pin "13"
-		)
 		(instances

Commit message: Rev2
Connections:
- net +5V: now also J1.1 (Pin_1); no longer J1.2 (Pin_2)
- net DCMotor/DIR1: now also IC1.J321 (38); no longer IC1.J118 (6)
- net DCMotor/DIR2: now also IC1.J320 (39); no longer IC1.J119 (7)
- net DCMotor/DIR3: now also IC1.J319 (40); no longer IC1.J120 (8)
- net DCMotor/DIR4: now also IC1.J318 (41); no longer IC1.J121 (9)
- net DCMotor/DIR5: now also IC1.J317 (42); no longer IC1.J122 (10)
- net DCMotor/PWM1: now also IC1.J326 (33); no longer IC1.J123 (11)
- net DCMotor/PWM2: now also IC1.J325 (34); no longer IC1.J124 (12)
- net DCMotor/PWM3: now also IC1.J324 (35); no longer IC1.J125 (13)
- net DCMotor/PWM4: now also IC1.J323 (36); no longer IC1.J126 (14)
- net DCMotor/PWM5: now also IC1.J322 (37); no longer IC1.J127 (15)
- net GND: now also J1.2 (Pin_2); no longer J1.1 (Pin_1)
- net Servo/Servo1: now also IC1.J123 (11); no longer IC1.J113 (1)
- net Servo/Servo2: now also IC1.J124 (12); no longer IC1.J114 (2)
- net Servo/Servo3: now also IC1.J125 (13); no longer IC1.J115 (3)
- net Servo/Servo4: now also IC1.J126 (14); no longer IC1.J116 (4)
- net Servo/Servo5: now also IC1.J127 (15); no longer IC1.J117 (5)
- net ~{EMS}_{INFO}: now also IC1.J128 (16); no longer IC1.J317 (42), J1.4 (Pin_4)
- net at IC1.J112 (0): now also J1.4 (Pin_4)
- net at J1.5 (Pin_5): now also IC1.J113 (1); no longer IC1.J318 (41)
- net at J1.6 (Pin_6): now also IC1.J114 (2); no longer IC1.J319 (40)
- net at J1.7 (Pin_7): now also IC1.J115 (3); no longer IC1.J320 (39)
- net at J1.8 (Pin_8): now also IC1.J116 (4); no longer IC1.J321 (38)
- net at J1.9 (Pin_9): now also IC1.J117 (5); no longer IC1.J322 (37)
- net at J1.10 (Pin_10): now also IC1.J118 (6); no longer IC1.J323 (36)
- net at J1.11 (Pin_11): now also IC1.J119 (7); no longer IC1.J324 (35)
- net at J1.12 (Pin_12): now also IC1.J120 (8); no longer IC1.J325 (34)
- net at J1.13 (Pin_13): now also IC1.J121 (9); no longer IC1.J326 (33)
- net at J1.14 (Pin_14): now also IC1.J122 (10); no longer IC1.J327 (26)
- no-connect marks 12 -> 11
Other:
- moved on the sheet: J1

Commit message: Rev1.2
Connections:
- net Servo/Servo1: now also IC1.J331 (18); no longer IC1.J123 (11)
- net Servo/Servo2: now also IC1.J330 (19); no longer IC1.J124 (12)
- net Servo/Servo3: now also IC1.J329 (20); no longer IC1.J125 (13)
- net Servo/Servo4: now also IC1.J328 (21); no longer IC1.J126 (14)
- net Servo/Servo5: now also IC1.J327 (26); no longer IC1.J127 (15)
