File: ActuatorPowerSupply.kicad_sch (KiCad schematic)
At the start: 24 parts, among them IC1 NCP3020ADR2G, Q1 IRFIZ24NPbF, Q2 VBZM630

Commit message: CircuitComplete
Parts:
- IC2: renamed from IC1; footprint SOIC127P600X175-8N -> SamacSys_Parts:SOIC127P600X175-8N
- renumbered C4 to C1, C5 to C2, C6 to C3, C3 to C4, C2 to C5, C1 to C6, R5 to R10, R6 to R11, R10 to R2, R2 to R4, R11 to R5, R4 to R6, R9 to R7, R7 to R8, R8 to R9
Connections:
- net VCC renamed +BATT
Other:
- moved on the sheet: C1, C2, C3, R1, R2, R3, R4, R5, R6, R7

Commit message: Rev1
Parts:
- removed L1: PDPMAA1712-101MP, original:PDPMAA1712-101MP, symbol Device:L
- removed Q2: VBZM630, Package_TO_SOT_THT:TO-220-3_Vertical, symbol original:VBZM630
- added L1: 60B104C, SamacSys_Parts:60B104C, symbol SamacSys_Parts:60B104C
- added Q15: NTA7002NT1G, SamacSys_Parts:SOT50P160X90-3N, symbol SamacSys_Parts:NTA7002NT1G
- added R62: 10k, Resistor_SMD:R_0603_1608Metric, symbol Device:R
- added U8: TSM3446CX6, SamacSys_Parts:SOT95P280X95-6N, symbol SamacSys_Parts:TSM3446CX6
Connections:
- net +7.5V: now also L1.2
- net GNDPWR: now also Q15.2 (D), U8.4 (SOURCE); no longer IC2.4 (GND)
- net at C7.2, IC2.6 (VSW), Q1.3 (S)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: now also L1.1, U8.1 (DRAIN_1), U8.2 (DRAIN_2), U8.5 (DRAIN_3), U8.6 (DRAIN_4)
- net at IC2.5 (LSDR), R9.1: now also U8.3 (GATE)
- new net: Q15.1 (G), R62.2
- new net: IC2.4 (GND), Q15.3 (S)
- new net MS: R62.1
Other:
- moved on the sheet: C8, R10, R11, R9

Commit message: Rev1
Parts:
- Q15: JLCPCB Parts# (none) -> C145524
Changed lines of the file:
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@@
 			)
 		)
+		(property "JLCPCB Parts#" ""
+			(at 110.49 101.6 0)
+			(effects
+				(font
+					(size 1.27 1.27)
+				)
+				(hide yes)
+			)
+		)
 		(pin "2"
 		)
@@
 			)
 		)
+		(property "JLCPCB Parts#" ""
+			(at 72.39 121.92 0)
+			(effects
+				(font
+					(size 1.27 1.27)
+				)
+				(hide yes)
+			)
+		)
 		(pin "2"
 		)
@@
 			)
 		)
+		(property "JLCPCB Parts#" ""
+			(at 59.69 115.57 0)
+			(effects
+				(font
+					(size 1.27 1.27)
+				)
+				(hide yes)
+			)
+		)
 		(pin "2"
 		)
@@
 			)
 		)
+		(property "JLCPCB Parts#" ""
+			(at 25.4 120.65 0)
+			(effects
+				(font
+					(size 1.27 1.27)
+				)
+				(hide yes)
+			)
+		)
 		(pin "1"
 		)
@@
 			)
 		)
+		(property "JLCPCB Parts#" ""
+			(at 231.14 99.06 0)
+			(effects
+				(font
+					(size 1.27 1.27)
+				)
+				(hide yes)
+			)
+		)
 		(pin "1"
 		)
@@
 			)
 		)
+		(property "JLCPCB Parts#" ""
+			(at 31.75 104.14 0)
+			(effects
+				(font
+					(size 1.27 1.27)
+				)
+				(hide yes)
+			)
+		)
 		(pin "2"
 		)
@@
 			)
 		)
+		(property "JLCPCB Parts#" ""
+			(at 190.5 72.39 0)
+			(effects
+				(font
+					(size 1.27 1.27)
+				)
+				(hide yes)
+			)
+		)
 		(instances
 			(project ""
@@
 			)
 		)
+		(property "JLCPCB Parts#" ""
+			(at 49.53 121.92 0)
+			(effects
+				(font
+					(size 1.27 1.27)
+				)
+				(hide yes)
+			)
+		)
 		(pin "2"
 		)
@@
 			)
 		)
+		(property "JLCPCB Parts#" ""
+			(at 139.7 74.93 0)
+			(effects
+				(font
+					(size 1.27 1.27)
+				)
+				(hide yes)
+			)
+		)
 		(pin "8"
 		)
@@
 			)
 		)
+		(property "JLCPCB Parts#" ""
+			(at 120.65 81.28 0)
+			(effects
+				(font
+					(size 1.27 1.27)
+				)
+				(hide yes)
+			)
+		)
 		(pin "2"
 		)
@@
 			)
 		)
+		(property "JLCPCB Parts#" ""
+			(at 186.69 83.82 0)
+			(effects
+				(font
+					(size 1.27 1.27)
+				)
+				(hide yes)
+			)
+		)
 		(pin "1"
 		)
@@
 			)
 		)
+		(property "JLCPCB Parts#" ""
+			(at 168.91 109.22 0)
+			(effects
+				(font
+					(size 1.27 1.27)
+				)
+				(hide yes)
+			)
+		)
 		(pin "2"
 		)
@@
 			)
 		)
+		(property "JLCPCB Parts#" ""
+			(at 243.84 95.25 0)
+			(effects
+				(font
+					(size 1.27 1.27)
+				)
+				(hide yes)
+			)
+		)
 		(pin "1"
 		)
@@
 			)
 		)
+		(property "JLCPCB Parts#" ""
+			(at 25.4 109.22 0)
+			(effects
+				(font
+					(size 1.27 1.27)
+				)
+				(hide yes)
+			)
+		)
 		(pin "2"
 		)
@@
 			)
 		)
+		(property "JLCPCB Parts#" ""
+			(at 195.58 77.47 0)
+			(effects
+				(font
+					(size 1.27 1.27)
+				)
+				(hide yes)
+			)
+		)
 		(pin "3"
 		)
@@
 			)
 		)
+		(property "JLCPCB Parts#" ""
+			(at 205.74 90.17 0)
+			(effects
+				(font
+					(size 1.27 1.27)
+				)
+				(hide yes)
+			)
+		)
 		(pin "2"
 		)
@@
 			)
 		)
+		(property "JLCPCB Parts#" ""
+			(at 100.33 81.28 0)
+			(effects
+				(font
+					(size 1.27 1.27)
+				)
+				(hide yes)
+			)
+		)
 		(pin "1"
 		)
@@
 			)
 		)
+		(property "JLCPCB Parts#" ""
+			(at 110.49 81.28 0)
+			(effects
+				(font
+					(size 1.27 1.27)
+				)
+				(hide yes)
+			)
+		)
 		(pin "1"
 		)
@@
 			)
 		)
+		(property "JLCPCB Parts#" ""
+			(at 25.4 97.79 0)
+			(effects
+				(font
+					(size 1.27 1.27)
+				)
+				(hide yes)
+			)
+		)
 		(pin "2"
 		)
@@
 			)
 		)
+		(property "JLCPCB Parts#" ""
+			(at 243.84 106.68 0)
+			(effects
+				(font
+					(size 1.27 1.27)
+				)
+				(hide yes)
+			)
+		)
 		(pin "1"
 		)
@@
 			)
 		)
+		(property "JLCPCB Parts#" ""
+			(at 60.96 121.92 0)
+			(effects
+				(font
+					(size 1.27 1.27)
+				)
+				(hide yes)
+			)
+		)
 		(pin "2"
 		)
@@
 			)
 		)
+		(property "JLCPCB Parts#" ""
+			(at 31.75 118.11 0)
+			(effects
+				(font
+					(size 1.27 1.27)
+				)
+				(hide yes)
+			)
+		)
 		(pin "2"
 		)
@@
 			)
 		)
+		(property "JLCPCB Parts#" " C145524"
+			(at 116.84 101.6 0)
+			(effects
+				(font
+					(size 1.27 1.27)
+				)
+				(hide yes)
+			)
+		)
 		(pin "3"
 		)
@@
 			)
 		)
+		(property "JLCPCB Parts#" ""
+			(at 25.4 137.16 0)
+			(effects
+				(font
+					(size 1.27 1.27)
+				)
+				(hide yes)
+			)
+		)
 		(pin "2"
 		)
@@
 			)
 		)
+		(property "JLCPCB Parts#" ""
+			(at 177.8 83.82 0)
+			(effects
+				(font
+					(size 1.27 1.27)
+				)
+				(hide yes)
+			)
+		)
 		(pin "1"
 		)
@@
 				(hide yes)
 			)
+		)
+		(property "JLCPCB Parts#" ""
+			(at 180.34 100.33 0)
+			(effects
+				(font
+					(size 1.27 1.27)
+				)
+				(hide yes)
+			)

Commit message: before elimination of J7
Parts:
- removed R10: 150k, Resistor_SMD:R_0603_1608Metric, symbol Device:R
- removed R11: 10k, Resistor_SMD:R_0603_1608Metric, symbol Device:R
- C2: value 33p -> 18p
- C3: value 1n -> 3.3n
- HS1: value Heatsink -> BPUE56-25; footprint original:BPUG56 -> original:BPUE56
- L1: footprint SamacSys_Parts:60B104C -> original:60B104C_correct
- R2: value 48 -> 18
- R3: value 220 -> 1.6k
- R4: value 2.2k -> 13k
- R5: value 330 -> 4.7k
- R6: value 16k -> 3k
- R7: value 16k -> 56k
- R9: value 27k -> 56k
- renumbered Q15 to Q1, Q1 to Q2, R8 to R10, R62 to R8, U8 to U1
Connections:
- net FB: no longer C2.1, R6.1
- net GNDPWR: now also C2.1, R6.1
Other:
- moved on the sheet: C2, C3, R6, R7

Commit message: gaber
Parts:
- IC2: JLCPCB Parts# (none) -> C457728
- Q2: JLCPCB Parts# (none) -> C537925
- U1: JLCPCB Parts# (none) -> C3290101
Changed lines of the file:
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@@
 			)
 		)
-		(property "JLCPCB Parts#" ""
+		(property "JLCPCB Parts#" "C457728"
 			(at 139.7 74.93 0)
 			(effects
@@
 			)
 		)
-		(property "JLCPCB Parts#" ""
+		(property "JLCPCB Parts#" " C537925"
 			(at 195.58 77.47 0)
 			(effects
@@
 			)
 		)
-		(property "JLCPCB Parts#" ""
+		(property "JLCPCB Parts#" "C3290101"
 			(at 180.34 100.33 0)
 			(effects
