File: SoftStart.kicad_sch (KiCad schematic)
At the start: 7 parts, among them IC6 D44H8, Q11 2SC2712-GR_TE85L,F, Q12 2SC2712-GR_TE85L,F

Commit message: Rev1
Parts:
- removed IC6: D44H8, SamacSys_Parts:TO270P460X1020X2008-3P, symbol SamacSys_Parts:D44H8
- added D10: 12V_Zener, Diode_SMD:D_SOD-323, symbol Device:D_Zener
- added Q2: IRFR014TRPBF-BE3, SamacSys_Parts:IRFR014TRPBFBE3, symbol SamacSys_Parts:IRFR014TRPBF-BE3
- R57: value 510 -> 2.2k
- R58: value 1.5 -> 1.3; footprint Resistor_SMD:R_0603_1608Metric -> Resistor_SMD:R_1206_3216Metric
Connections:
- net -BATT: now also D10.2 (A)
- net GNDPWR: now also Q2.2
- net at Q12.1 (BASE), R58.1: now also Q2.3
- net at Q11.3 (COLLECTOR), Q12.3 (COLLECTOR), R57.2: now also D10.1 (K), Q2.1
- net LOGPWR renamed SAFE_+BATT
Other:
- moved on the sheet: R58

Commit message: Rev1
Parts:
- D10: JLCPCB Parts# (none) -> C19077447
- Q11, Q12: JLCPCB Parts# (none) -> C83447

Commit message: before elimination of J7
Parts:
- renumbered D10 to D8, Q2 to Q12, Q12 to Q13, R55 to R54, R56 to R55, R57 to R56, R58 to R57

Commit message: gaber
Parts:
- Q12: JLCPCB Parts# (none) -> C3290995

Commit message: add order information
Parts:
- R57: JLCPCB Parts# (none) -> C4048845
